File: SqueezeAMPagain/SqueezeAMPagain.kicad_pcb (KiCad board)
At the start: 2 copper layers, 67 parts, among them J1 Conn_01x02_Pin, J2 Conn_01x02_Pin, J3 Raspberry_Pi_2_3, J4 Conn_01x06_Pin, Q1 Q_NPN_BEC, Q2 PMOS, U1 TAS5756M, U2 RaspberryPi_Pico_W, U4 ESP32-WROVER-E

Commit message: Update .gitignore, L_Radial_D12.0mm_P5+6+7.00mm_Fastron_11P.kicad_mod, SqueezeAMPagain.kicad_pcb, and 13 more files
Parts:
- added C42: 100n, Capacitor_SMD:C_0603_1608Metric, F.Cu at (153.0, 53.2)
- added C43: 10u/50V, Capacitor_SMD:C_1206_3216Metric, F.Cu at (141.0, 71.5)
- added C44: 100n, Capacitor_SMD:C_0603_1608Metric, F.Cu at (141.7, 69.0)
- added C45: 10u/50V, Capacitor_SMD:C_1206_3216Metric, F.Cu at (155.5, 70.5)
- added C46: 100n, Capacitor_SMD:C_0603_1608Metric, F.Cu at (70.2, 34.5)
- added C47: 2.2u/25V, Capacitor_SMD:C_0805_2012Metric, F.Cu at (70.0, 32.0)
- added C48: 100n, Capacitor_SMD:C_0603_1608Metric, F.Cu at (75.5, 27.3)
- added C49: 0.01 μF low ESR, Capacitor_SMD:C_0603_1608Metric, F.Cu at (174.2, 95.8)
- added C50: 100n, Capacitor_SMD:C_0603_1608Metric, F.Cu at (159.0, 93.0)
- added C51: 150p, Capacitor_SMD:C_0603_1608Metric, F.Cu at (161.2, 93.0)
- added C52: 100n, Capacitor_SMD:C_0603_1608Metric, F.Cu at (109.4, 34.5)
- added C53: 100n, Capacitor_SMD:C_0603_1608Metric, F.Cu at (58.7, 77.0)
- added C54: 470u/35V rad, THT, Capacitor_THT:CP_Radial_D8.0mm_P5.00mm, F.Cu at (145.8, 73.0)
- added C55: 100n, Capacitor_SMD:C_0603_1608Metric, F.Cu at (61.2, 72.0)
- added C56: 2.2u/25V, Capacitor_SMD:C_0805_2012Metric, F.Cu at (151.6, 97.0)
- added C57: 100n, Capacitor_SMD:C_0603_1608Metric, F.Cu at (137.7, 82.5)
- added C58: 2.2u/25V, Capacitor_SMD:C_0603_1608Metric, F.Cu at (160.7, 78.5)
- added C59: 100n, Capacitor_SMD:C_0603_1608Metric, F.Cu at (184.8, 76.7)
- added C60: 10u/50V, Capacitor_SMD:C_1206_3216Metric, F.Cu at (189.6, 80.5)
- added C61: 2.2u/25V, Capacitor_SMD:C_0805_2012Metric, F.Cu at (184.8, 79.2)
- added C62: 2.2u/25V, Capacitor_SMD:C_0805_2012Metric, F.Cu at (96.0, 63.5)
- added C63: 100n, Capacitor_SMD:C_0603_1608Metric, F.Cu at (105.3, 38.8)
- added C64: 100n, Capacitor_SMD:C_0603_1608Metric, F.Cu at (114.5, 36.8)
- added C65: 100n, Capacitor_SMD:C_0603_1608Metric, F.Cu at (118.0, 36.2)
- added C66: 100n, Capacitor_SMD:C_0603_1608Metric, F.Cu at (109.6, 38.5)
- added C67: 100n, Capacitor_SMD:C_0603_1608Metric, F.Cu at (105.1, 34.5)
- added C68: 100n, Capacitor_SMD:C_0603_1608Metric, F.Cu at (114.5, 34.5)
- added C69: 100n, Capacitor_SMD:C_0603_1608Metric, F.Cu at (118.0, 34.5)
- added C70: 470u, Capacitor_THT:CP_Radial_D10.0mm_P5.00mm_P7.50mm, F.Cu at (135.5, 36.5)
- added C71: 470u, Capacitor_SMD:CP_Elec_6.3x3.9, F.Cu at (148.0, 70.2)
- added C72: 470u, Capacitor_THT:CP_Radial_D10.0mm_P5.00mm_P7.50mm, F.Cu at (85.5, 48.0)
- added D1: D_Schottky, Diode_SMD:D_0603_1608Metric, F.Cu at (73.7, 30.0)
- added D2: SS34, Diode_SMD:D_0805_2012Metric, F.Cu at (169.9, 96.1)
- added D3: D_Schottky, Diode_SMD:D_0805_2012Metric, F.Cu at (169.9, 99.2)
- added J5: USB_B_Micro, Connector_USB:USB_Micro-B_Wuerth_629105150521_CircularHoles, F.Cu at (82.0, 24.5)
- added J6: Conn_01x02_Pin, Connector_Phoenix_MC:PhoenixContact_MC_1,5_2-G-3.5_1x02_P3.50mm_Horizontal, F.Cu at (150.0, 29.5)
- added J7: Barrel_Jack_Switch_MountingPin, Connector_BarrelJack:BarrelJack_CUI_PJ-079BH_Horizontal, F.Cu at (143.9, 31.0)
- added J8: Conn_02x08_Odd_Even, Connector_IDC:IDC-Header_2x08_P2.54mm_Vertical, F.Cu at (134.3, 109.5)
- added J9: Conn_01x06_Pin, Connector_PinHeader_2.54mm:PinHeader_1x06_P2.54mm_Vertical, F.Cu at (68.5, 56.0)
- added JP3: RPP, Jumper:SolderJumper-2_P1.3mm_Open_RoundedPad1.0x1.5mm, F.Cu at (145.5, 35.5)
- added JP4: P On, Jumper:SolderJumper-2_P1.3mm_Open_RoundedPad1.0x1.5mm, F.Cu at (150.4, 52.5)
- added JP5: LV On, Jumper:SolderJumper-2_P1.3mm_Open_RoundedPad1.0x1.5mm, F.Cu at (150.0, 61.1)
- added JP6: Mono, Jumper:SolderJumper-2_P1.3mm_Open_RoundedPad1.0x1.5mm, F.Cu at (129.3, 66.5)
- added JP7: Mono, Jumper:SolderJumper-2_P1.3mm_Open_RoundedPad1.0x1.5mm, F.Cu at (129.2, 69.0)
- added L10: 680nH, Inductor_SMD:L_0805_2012Metric, F.Cu at (73.9, 34.0)
- added L11: 22uH, Inductor_SMD:L_SXN_SMDRI74, F.Cu at (151.5, 89.5)
- added L12: 680nH, Inductor_SMD:L_0805_2012Metric, F.Cu at (150.5, 65.5)
- added L8: 4.7uH/3.0A, Inductor:L_Radial_D12.0mm_P5+6+7.00mm_Fastron_11P, F.Cu at (148.0, 41.5)
- added L9: 4.7uH/3.0A, Inductor:L_Radial_D12.0mm_P5+6+7.00mm_Fastron_11P, F.Cu at (144.0, 59.0)
- added NT1: NetTie_2, NetTie:NetTie-2_SMD_Pad2.0mm, B.Cu at (152.5, 36.0)
- added NT2: NetTie_2, NetTie:NetTie-2_SMD_Pad2.0mm, B.Cu at (144.0, 56.0)
- added Q3: PMOS, Package_DFN_QFN:Diodes_UDFN2020-6_Type-F, F.Cu at (150.5, 35.5)
- added Q4: Q_NPN_BEC, Package_TO_SOT_SMD:SOT-23, F.Cu at (73.6, 45.5)
- added Q5: Q_NPN_BEC, Package_TO_SOT_SMD:SOT-23, F.Cu at (79.4, 46.0)
- added Q6: Q_NPN_BEC, Package_TO_SOT_SMD:SOT-23, F.Cu at (157.6, 64.5)
- added Q7: PMOS, Package_DFN_QFN:Diodes_UDFN2020-6_Type-F, F.Cu at (156.5, 60.5)
- added R10: 33, Resistor_SMD:R_0402_1005Metric, F.Cu at (106.0, 79.0)
- added R11: 33, Resistor_SMD:R_0402_1005Metric, F.Cu at (115.5, 79.0)
- added R12: 10k, Resistor_SMD:R_0603_1608Metric, F.Cu at (145.1, 87.3)
- added R13: 5.9k, Resistor_SMD:R_0603_1608Metric, F.Cu at (145.0, 91.0)
- added R14: 549R, Resistor_SMD:R_0603_1608Metric, F.Cu at (143.0, 91.0)
- added R15: 10k, Resistor_SMD:R_0603_1608Metric, F.Cu at (153.2, 60.0)
- added R16: 10k, Resistor_SMD:R_0603_1608Metric, F.Cu at (154.2, 64.5)
- added R17: 150k, Resistor_SMD:R_0603_1608Metric, F.Cu at (148.0, 35.8)
- added R18: 150k, Resistor_SMD:R_0603_1608Metric, F.Cu at (153.5, 62.3)
- added R19: 10k, Resistor_SMD:R_0603_1608Metric, F.Cu at (159.7, 82.0)
- added R20: 10k, Resistor_SMD:R_0603_1608Metric, F.Cu at (137.2, 88.5)
- added R21: 49.9k, Resistor_SMD:R_0603_1608Metric, F.Cu at (129.2, 64.5)
- added R4: 150k, Resistor_SMD:R_0603_1608Metric, F.Cu at (147.4, 52.2)
- added R5: 10k, Resistor_SMD:R_0603_1608Metric, F.Cu at (153.0, 35.7)
- added R6: 10k, Resistor_SMD:R_0603_1608Metric, F.Cu at (69.5, 45.7)
- added R7: 10k, Resistor_SMD:R_0603_1608Metric, F.Cu at (76.5, 45.0)
- added R8: 33, Resistor_SMD:R_0402_1005Metric, F.Cu at (112.0, 79.0)
- added R9: 33, Resistor_SMD:R_0402_1005Metric, F.Cu at (110.5, 79.0)
- added U3: CP2102N-Axx-xQFN28, Package_DFN_QFN:QFN-28-1EP_5x5mm_P0.5mm_EP3.35x3.35mm, F.Cu at (75.7, 35.5)
- added U5: TPS5430DDA, Package_SO:TI_SO-PowerPAD-8_ThermalVias, F.Cu at (160.8, 87.6)
- added U6: TSOP21xx, OptoDevice:Vishay_MOLD-3Pin, F.Cu at (159.9, 108.0)
- C1, C10, C11, C12, C14, C15, C16, C17, C18, C36, C40: footprint Capacitor_SMD:C_0603_1608Metric -> Capacitor_SMD:C_0805_2012Metric
- C20, C21, C23, C25, C27: value 22u/35V -> 10u/50V
- C28, C29, C30, C31: footprint Capacitor_SMD:CP_Elec_6.3x3.9 -> Capacitor_THT:CP_Radial_D10.0mm_P5.00mm_P7.50mm
- C3, C5, C7, C9: value 0.68uF/50V -> 470n/50V; footprint Capacitor_SMD:C_0603_1608Metric -> Capacitor_SMD:C_0805_2012Metric
- C38: value 2.2u/25V -> 10u/50V; footprint Capacitor_SMD:C_0603_1608Metric -> Capacitor_SMD:C_1206_3216Metric
- J4: footprint Connector_PinHeader_2.54mm:PinHeader_1x06_P2.54mm_Horizontal -> Connector_PinHeader_2.54mm:PinHeader_1x06_P2.54mm_Vertical
- JP1, JP2: value SolderJumper_3_Bridged12 -> Mono; footprint Jumper:SolderJumper-3_P1.3mm_Bridged12_RoundedPad1.0x1.5mm -> Jumper:SolderJumper-2_P1.3mm_Open_RoundedPad1.0x1.5mm
- L1, L2, L3, L4: footprint Inductor_SMD:L_7.3x7.3_H3.5 -> Inductor:L_Radial_D12.0mm_P5+6+7.00mm_Fastron_11P
- L5, L6, L7: value L -> 680nH; footprint Inductor_SMD:L_0603_1608Metric -> Inductor_SMD:L_0805_2012Metric
- moved Q2 65.8 mm to (145.0, 52.5), turned to 180 degrees
- moved C31 61.8 mm to (83.5, 34.5), turned to 0 degrees
- moved C38 58.5 mm to (155.5, 54.0), turned to 90 degrees
- moved H1 56.4 mm to (70.5, 23.5)
- moved C30 53.5 mm to (91.5, 27.0), turned to 0 degrees
- moved R3 52.2 mm to (151.3, 59.5)
- moved Q1 51.9 mm to (151.5, 56.6), turned to 90 degrees
- moved C28 48.2 mm to (129.0, 27.0), turned to 0 degrees
- moved C29 46.3 mm to (134.0, 48.0), turned to 0 degrees
- moved H3 44.5 mm to (158.5, 25.0)
- moved J4 40.4 mm to (127.0, 84.5)
- moved R2 39.5 mm to (139.3, 78.0)
- moved U2 38.4 mm to (76.6, 86.5)
- moved JP2 29.6 mm to (120.8, 55.5)
- moved R1 27.6 mm to (123.0, 101.2), turned to 90 degrees
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Connections:
- net /esp/EN/~{RESET} renamed /USB-Uart/EN/~{RESET}
- C22 pad 1: +3V3 -> +3.3V
- C3 pad 2: GND1 -> PGND
- C38 pad 1: /Amp/GVDD_REG -> VIN
- C38 pad 2: PGND -> Net-(Q1-E)
- C40 pad 1: +3V3 -> +3.3V
- C5 pad 2: GND1 -> PGND
- C7 pad 2: GND1 -> PGND
- C9 pad 2: GND1 -> PGND
- J3 pad 12: unconnected-(J3-GPIO18/PWM0-Pad12) -> /Pi/BCLK
- J3 pad 3: unconnected-(J3-SDA/GPIO2-Pad3) -> /Pi/SDA
- J3 pad 32: unconnected-(J3-PWM0/GPIO12-Pad32) -> /Pi/PWM
- J3 pad 35: unconnected-(J3-GPIO19/MISO1-Pad35) -> /Pi/LRCLK
- J3 pad 40: unconnected-(J3-GPIO21/SCLK1-Pad40) -> /Pi/DATA
- J3 pad 5: unconnected-(J3-SCL/GPIO3-Pad5) -> /Pi/SCL
- J4 pad 5: +3V3 -> +3.3V
- JP1 pad 1: GND -> /Amp/SpeakerChannelA-/Amp_out
- JP1 pad 2: Net-(JP1-C) -> /Amp/SpeakerChannelA+/Amp_out
- JP2 pad 1: GND -> /Amp/SpeakerChannelB-/Amp_out
- JP2 pad 2: Net-(JP2-C) -> /Amp/SpeakerChannelB+/Amp_out
- Q1 pad 2: unconnected-(Q1-E-Pad2) -> Net-(Q1-E)
- Q1 pad 3: unconnected-(Q1-C-Pad3) -> Net-(Q1-C)
- Q2 pad 1: unconnected-(Q2-D-Pad1) -> Net-(JP4-B)
- Q2 pad 2: unconnected-(Q2-G-Pad2) -> Net-(Q1-C)
- Q2 pad 3: unconnected-(Q2-S-Pad3) -> VIN
- R1 pad 1: +3V3 -> +3.3V
- R2 pad 1: unconnected-(R2-Pad1) -> /Power/PON
- R3 pad 1: unconnected-(R3-Pad1) -> Net-(Q1-B)
- R3 pad 2: unconnected-(R3-Pad2) -> Net-(Q1-E)
- U1 pad 20: Net-(JP1-C) -> GND
- U1 pad 22: /Amp/MCLK -> Net-(U1-MCLK)
- U1 pad 23: /Amp/SCLK -> Net-(U1-SCLK)
- U1 pad 24: /Amp/SDIN -> Net-(U1-SDIN)
- U1 pad 25: /Amp/LRCLK/FS -> Net-(U1-LRCK/FS)
- U1 pad 26: Net-(JP2-C) -> GND
- U2 pad 1: unconnected-(U2-GPIO0-Pad1) -> /USB-Uart/RX
- U2 pad 16: unconnected-(U2-GPIO12-Pad16) -> /USB-Uart/BOOT
- U2 pad 19: unconnected-(U2-GPIO14-Pad19) -> /Amp/SCLK
- U2 pad 2: unconnected-(U2-GPIO1-Pad2) -> /USB-Uart/TX
- U2 pad 20: unconnected-(U2-GPIO15-Pad20) -> /Amp/SDIN
- U2 pad 4: unconnected-(U2-GPIO2-Pad4) -> /FPConnector/SCK
- U2 pad 5: unconnected-(U2-GPIO3-Pad5) -> /FPConnector/MOSI
- U2 pad 6: unconnected-(U2-GPIO4-Pad6) -> /FPConnector/MISO
- U2 pad 7: unconnected-(U2-GPIO5-Pad7) -> /FPConnector/CS
- U4 pad 10: /esp/I2S-WS -> /Amp/LRCLK/FS
- U4 pad 11: /esp/D/C -> /FPConnector/D/C
- U4 pad 12: unconnected-(U4-ADC2_CH7/GPIO27-Pad12) -> /Power/PON
- U4 pad 2: +3V3 -> +3.3V
- U4 pad 24: /esp/IO2 -> /FPConnector/RESET
- U4 pad 25: /esp/GPIO0/BOOT -> /USB-Uart/BOOT
- U4 pad 26: /esp/IO4 -> /FPConnector/IO4
- U4 pad 29: /esp/VSPICS0 -> /FPConnector/CS
- U4 pad 30: /esp/VSPICLK -> /FPConnector/SCK
- U4 pad 31: /esp/VSPIQ -> /FPConnector/MISO
- U4 pad 34: /esp/RX -> /USB-Uart/TX
- U4 pad 35: /esp/TX -> /USB-Uart/RX
- U4 pad 37: /esp/VSPID -> /FPConnector/MOSI
- U4 pad 4: unconnected-(U4-SENSOR_VP/GPIO36/ADC1_CH0-Pad4) -> /Amp/~{SPK_FAULT}
- U4 pad 5: unconnected-(U4-SENSOR_VN/GPIO39/ADC1_CH3-Pad5) -> /FPConnector/IO3
- U4 pad 6: unconnected-(U4-GPIO34/ADC1_CH6-Pad6) -> /FPConnector/IO2
- U4 pad 7: unconnected-(U4-GPIO35/ADC1_CH7-Pad7) -> /FPConnector/IO1
- U4 pad 9: /esp/I2S-CLK -> /Amp/SCLK
Routing:
- net /Amp/SCL: track 0.00 -> 41.0 mm
- net /Amp/SDA: track 0.00 -> 37.7 mm
- net +3.3V: track 34.0 -> 0.00 mm, vias 6 -> 0
- net Net-(JP6-A): track 26.8 -> 0.00 mm
- net GNDA: track 4.51 -> 27.5 mm
- net Net-(U1-SPK_GAIN/FREQ): track 0.00 -> 18.7 mm
- net /Amp/SpeakerChannelB+/Amp_out: track 15.2 -> 0.00 mm
- net Net-(U1-MCLK): track 0.00 -> 13.3 mm
- net Net-(U1-SCLK): track 0.00 -> 11.6 mm
- net Net-(U1-AVDD): track 0.00 -> 10.7 mm
- net Net-(U1-SDIN): track 0.00 -> 10.1 mm
- net /Amp/GVDD_REG: track 5.86 -> 15.1 mm
- net Net-(JP2-C): track 8.58 -> 0.00 mm
- net Net-(U1-SPK_INA-): track 0.97 -> 9.55 mm
- net /Amp/SpeakerChannelA+/Cboot: track 0.00 -> 7.67 mm
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- added copper zone on B.Cu, net /Amp/SPK_A+
- added copper zone on F.Cu, net /Amp/SPK_A+
- added copper zone on B.Cu, net /Amp/SPK_A-
- added copper zone on F.Cu, net /Amp/SPK_A-
- added copper zone on B.Cu, net /Amp/SPK_B+
- added copper zone on F.Cu, net /Amp/SPK_B+
- added copper zone on B.Cu, net /Amp/SPK_B-
- added copper zone on F.Cu, net /Amp/SPK_B-
- added copper zone on F.Cu, net PGND
Other:
- board outline added: 109.5 x 108 mm

Commit message: Update SqueezeAMPagain.kicad_pcb, SqueezeAMPagain.kicad_prl, USB-Uart.kicad_sch, and 4 more files
Parts:
- removed C2, C4, C6, C8: 0.22uF/50V, Capacitor_SMD:C_0603_1608Metric
- removed L10, L12, L5, L6, L7: 680nH, Inductor_SMD:L_0805_2012Metric
- added C41: 220n, Capacitor_SMD:C_0805_2012Metric, F.Cu at (109.5, 55.5)
- added C73: 220n, Capacitor_SMD:C_0805_2012Metric, F.Cu at (102.0, 57.5)
- added C74: 220n, Capacitor_SMD:C_0805_2012Metric, F.Cu at (116.5, 55.5)
- added C75: 220n, Capacitor_SMD:C_0805_2012Metric, F.Cu at (122.5, 58.5)
- added C76: 100n, Capacitor_SMD:C_0603_1608Metric, F.Cu at (69.3, 37.5)
- added C77: 100n, Capacitor_SMD:C_0603_1608Metric, F.Cu at (64.5, 39.0)
- added C78: 2.2u/25V, Capacitor_SMD:C_0805_2012Metric, F.Cu at (63.5, 27.5)
- added C79: 2.2u/25V, Capacitor_SMD:C_0805_2012Metric, F.Cu at (64.0, 30.5)
- added C80: 100n, Capacitor_SMD:C_0603_1608Metric, F.Cu at (61.7, 33.5)
- added FB1: 600Ω@100MHz 500mA, Inductor_SMD:L_0805_2012Metric, F.Cu at (185.9, 67.5)
- added FB2: 600Ω@100MHz 500mA, Inductor_SMD:L_0805_2012Metric, F.Cu at (142.0, 75.5)
- added FB3: 600Ω@100MHz 500mA, Inductor_SMD:L_0805_2012Metric, F.Cu at (100.4, 71.5)
- added FB4: 600Ω@100MHz 500mA, Inductor_SMD:L_0805_2012Metric, F.Cu at (96.4, 72.5)
- added FB5: 600Ω@100MHz 500mA, Inductor_SMD:L_0805_2012Metric, F.Cu at (160.4, 68.5)
- added FB6: 600Ω@100MHz 500mA, Inductor_SMD:L_0805_2012Metric, F.Cu at (76.4, 30.0)
- added R22: 33, Resistor_SMD:R_0402_1005Metric, F.Cu at (113.5, 79.5)
- added R23: 33, Resistor_SMD:R_0402_1005Metric, F.Cu at (108.5, 79.5)
- added R24: 33, Resistor_SMD:R_0402_1005Metric, F.Cu at (117.5, 79.0)
- added R25: 33, Resistor_SMD:R_0402_1005Metric, F.Cu at (107.0, 79.0)
- added R26: 33, Resistor_SMD:R_0402_1005Metric, F.Cu at (119.0, 79.5)
- added R27: 10k, Resistor_SMD:R_0603_1608Metric, F.Cu at (100.2, 73.5)
- added R28: 10k, Resistor_SMD:R_0603_1608Metric, F.Cu at (100.0, 75.0)
- added R29: 10k, Resistor_SMD:R_0603_1608Metric, F.Cu at (64.2, 35.5)
- added R30: 10k, Resistor_SMD:R_0603_1608Metric, F.Cu at (69.8, 29.0)
- added R31: 10k, Resistor_SMD:R_0603_1608Metric, F.Cu at (66.0, 33.0)
- added U7: AMS1117-3.3, Package_TO_SOT_SMD:SOT-223-3_TabPin2, F.Cu at (62.9, 44.0)
- D2: footprint Diode_SMD:D_0805_2012Metric -> Diode_SMD:D_SMA
- moved C53 32.6 mm to (90.7, 71.0)
- moved C55 29.5 mm to (90.7, 73.5)
- moved R11 22.5 mm to (94.0, 85.5), turned to 0 degrees
- moved C60 22.1 mm to (199.0, 100.5)
- moved R8 18.0 mm to (94.0, 79.5), turned to 0 degrees
- moved R9 16.7 mm to (94.0, 81.5), turned to 0 degrees
- moved R10 12.8 mm to (94.0, 83.5), turned to 0 degrees
Connections:
- net /Amp/SCL renamed /SCL
- net /Amp/SDA renamed /SDA
- D3 pad 2: /esp/TDO -> /Power/~{WAKE_DETECT}
- R10 pad 1: /USB-Uart/BOOT -> /Amp/SDIN
- R10 pad 2: Net-(U1-MCLK) -> Net-(U2-GPIO15)
- R11 pad 2: Net-(U1-LRCK/FS) -> Net-(U2-GPIO13)
- R20 pad 2: /esp/TDO -> /Power/~{WAKE_DETECT}
- R8 pad 1: /Amp/SDIN -> /USB-Uart/BOOT
- R8 pad 2: Net-(U1-SDIN) -> Net-(U2-GPIO12)
- R9 pad 2: Net-(U1-SCLK) -> Net-(U2-GPIO14)
- U1 pad 22: Net-(U1-MCLK) -> /USB-Uart/BOOT
- U1 pad 23: Net-(U1-SCLK) -> /Amp/SCLK
- U1 pad 24: Net-(U1-SDIN) -> /Amp/SDIN
- U1 pad 25: Net-(U1-LRCK/FS) -> /Amp/LRCLK/FS
- U2 pad 16: /USB-Uart/BOOT -> Net-(U2-GPIO12)
- U2 pad 17: unconnected-(U2-GPIO13-Pad17) -> Net-(U2-GPIO13)
- U2 pad 19: /Amp/SCLK -> Net-(U2-GPIO14)
- U2 pad 20: /Amp/SDIN -> Net-(U2-GPIO15)
- U3 pad 6: unconnected-(U3-VDD-Pad6) -> Net-(U3-VDD)
- U3 pad 7: unconnected-(U3-VREGIN-Pad7) -> V_{USB}
- U3 pad 8: V_{USB} -> Net-(U3-VBUS)
- U4 pad 10: /Amp/LRCLK/FS -> Net-(U4-DAC_1/ADC2_CH8/GPIO25)
- U4 pad 25: /USB-Uart/BOOT -> Net-(U4-GPIO0/BOOT/ADC2_CH1)
- U4 pad 8: /Amp/SDIN -> Net-(U4-32K_XP/GPIO32/ADC1_CH4)
- U4 pad 9: /Amp/SCLK -> Net-(U4-32K_XN/GPIO33/ADC1_CH5)
- U6 pad 2: unconnected-(U6-Vs-Pad2) -> +3.3V
Routing:
- net Net-(U1-MCLK): track 13.3 -> 0.00 mm
- net /USB-Uart/BOOT: track 0.00 -> 13.3 mm
- net Net-(U1-SCLK): track 11.6 -> 0.00 mm
- net /Amp/SCLK: track 0.00 -> 11.6 mm
- net Net-(U1-SDIN): track 10.1 -> 0.00 mm
- net /Amp/SDIN: track 0.00 -> 10.1 mm
- net Net-(U1-LRCK/FS): track 5.55 -> 0.00 mm
- net /Amp/LRCLK/FS: track 0.00 -> 5.55 mm

Commit message: Update SqueezeAMPagain.kicad_pcb, project.db, power.kicad_sch, and 1 more file
Parts:
- added C2: 100n, Capacitor_SMD:C_0603_1608Metric, F.Cu at (175.0, 93.5)
- added C4: 1n, Capacitor_SMD:C_0603_1608Metric, F.Cu at (178.1, 93.0)
- added C6: 100n, Capacitor_SMD:C_0603_1608Metric, F.Cu at (190.0, 87.3)
- added C8: 220u/10V, Capacitor_THT:CP_Radial_D10.0mm_P2.50mm_P5.00mm, F.Cu at (156.8, 85.4)
- C41, C73, C74, C75: footprint Capacitor_SMD:C_0805_2012Metric -> Capacitor_SMD:C_0603_1608Metric
- C49: value 0.01 μF low ESR -> 10nF 78mOhm
- C54: value 470u/35V rad, THT -> 220u/10V; footprint Capacitor_THT:CP_Radial_D8.0mm_P5.00mm -> Capacitor_THT:CP_Radial_D10.0mm_P2.50mm_P5.00mm
- C58: footprint Capacitor_SMD:C_0603_1608Metric -> Capacitor_SMD:C_0805_2012Metric
- C71: value 470u -> 100u; footprint Capacitor_SMD:CP_Elec_6.3x3.9 -> Capacitor_SMD:C_1206_3216Metric
- D2: value SS34 -> SS34 550mV 2A
- L11: value 22uH -> 33uH 120mOhm
- R12: value 10k -> 22k
- R13: value 5.9k -> 13k
- R14: value 549R -> 560R
- moved C45 42.6 mm to (195.0, 86.5), turned to -90 degrees
- moved R14 38.7 mm to (181.5, 94.5)
- moved R13 36.5 mm to (181.5, 91.5), turned to 0 degrees
- moved R12 33.2 mm to (178.0, 91.5)
- moved C58 32.9 mm to (192.5, 87.0), turned to -90 degrees
- moved FB5 32.8 mm to (192.5, 75.4), turned to -90 degrees
- moved C54 29.6 mm to (169.0, 91.4), turned to -90 degrees
- moved C71 28.3 mm to (170.0, 52.5)
- moved L11 24.9 mm to (175.5, 82.7), turned to -90 degrees
- moved C57 24.1 mm to (159.5, 92.7), turned to -90 degrees
- moved U5 23.3 mm to (184.1, 87.3)
- moved D2 21.0 mm to (184.0, 80.5), turned to -90 degrees
- moved C51 20.3 mm to (181.6, 93.0)
- moved D3 19.9 mm to (150.5, 95.0)
- moved C61 19.7 mm to (204.6, 78.5)
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Connections:
- C71 pad 1: +3.3V -> unconnected-(C71-Pad1)
- C71 pad 2: GND -> unconnected-(C71-Pad2)

Commit message: Update SqueezeAMPagain.kicad_pcb, SqueezeAMPagain.kicad_sch, USB-Uart.kicad_sch, and 4 more files
Parts:
- removed D1: D_Schottky, Diode_SMD:D_0603_1608Metric
- added C81: 100u, Capacitor_SMD:C_1206_3216Metric, F.Cu at (40.3, 27.1)
- added C82: 100u, Capacitor_SMD:C_1206_3216Metric, F.Cu at (40.3, 30.4)
- added D4: B5819W, Diode_SMD:D_SOD-123, F.Cu at (61.0, 24.0)
- added JP10: SolderJumper_2_Open, Jumper:SolderJumper-2_P1.3mm_Open_RoundedPad1.0x1.5mm, F.Cu at (92.3, 68.5)
- added JP8: SolderJumper_2_Open, Jumper:SolderJumper-2_P1.3mm_Open_RoundedPad1.0x1.5mm, F.Cu at (92.3, 65.5)
- added JP9: SolderJumper_2_Bridged, Jumper:SolderJumper-2_P1.3mm_Bridged_RoundedPad1.0x1.5mm, F.Cu at (92.3, 62.5)
- added Q8: AO3401A, Package_TO_SOT_SMD:SOT-23, F.Cu at (158.9, 35.6)
- added Q9: AO3401A, Package_TO_SOT_SMD:SOT-23, F.Cu at (160.0, 48.1)
- added R32: 22k, Resistor_SMD:R_0603_1608Metric, F.Cu at (89.5, 68.8)
- added R33: 75k, Resistor_SMD:R_0603_1608Metric, F.Cu at (89.5, 62.0)
- D3: value D_Schottky -> B5819W; footprint Diode_SMD:D_0805_2012Metric -> Diode_SMD:D_SOD-123
- Q2, Q3, Q7: value PMOS -> AO3401A; footprint Package_DFN_QFN:Diodes_UDFN2020-6_Type-F -> Package_TO_SOT_SMD:SOT-23
- R100: value 750k -> 39k
- R101: value 150k -> 15k
- moved Q7 22.8 mm to (175.6, 73.0)
- moved Q2 15.0 mm to (160.0, 52.1), turned to -90 degrees
- moved R17 13.1 mm to (159.2, 42.5), turned to 0 degrees
- moved R4 13.0 mm to (160.2, 55.0), turned to 0 degrees
- moved JP3 12.0 mm to (157.0, 32.0), turned to 180 degrees
- moved JP4 12.0 mm to (159.3, 44.5), turned to 180 degrees
- moved Q3 9.43 mm to (158.9, 39.7), turned to -90 degrees
- moved Q1 8.72 mm to (160.0, 58.5)
- moved R5 8.43 mm to (160.5, 31.8)
- moved R100 5.61 mm to (89.5, 65.3), turned to -90 degrees
- moved C38 2.50 mm to (155.5, 56.5)
Connections:
- Q2 pad 1: Net-(JP4-B) -> Net-(Q1-C)
- Q2 pad 2: Net-(Q1-C) -> Net-(JP4-B)
- Q3 pad 1: Net-(J6-Pin_2) -> Net-(Q3-G)
- Q3 pad 2: Net-(Q3-G) -> Net-(JP3-B)
- Q3 pad 3: Net-(JP3-B) -> Net-(J6-Pin_2)
- Q7 pad 1: Net-(JP5-B) -> Net-(D3-K)
- Q7 pad 2: Net-(D3-K) -> Net-(JP5-B)
- R100 pad 1: Net-(U1-SPK_GAIN/FREQ) -> Net-(JP8-A)
- R101 pad 2: Net-(U1-SPK_GAIN/FREQ) -> Net-(JP10-B)
- U1 pad 9: Net-(U1-SPK_GAIN/FREQ) -> Net-(JP10-B)
Routing:
- net Net-(U1-SPK_GAIN/FREQ): track 18.7 -> 0.00 mm
- net Net-(JP10-B): track 0.00 -> 18.7 mm

Commit message: Update SqueezeAMPagain.kicad_pcb, SqueezeAMPagain.kicad_pro, amp.kicad_sch, and 2 more files
Parts:
- removed C71, C81: 100u, Capacitor_SMD:C_1206_3216Metric
- removed FB2: 600Ω@100MHz 500mA, Inductor_SMD:L_0805_2012Metric
- removed Q2: AO3401A, Package_TO_SOT_SMD:SOT-23
- added C83: 100u / 6.3V, Capacitor_SMD:C_1206_3216Metric, F.Cu at (147.0, 87.3)
- added FB7: 600Ω@100MHz 500mA, Inductor_SMD:L_0805_2012Metric, F.Cu at (155.8, 62.2)
- added JP11: Mono, Jumper:SolderJumper-2_P1.3mm_Open_RoundedPad1.0x1.5mm, F.Cu at (129.1, 71.8)
- added JP12: SolderJumper_2_Bridged, Jumper:SolderJumper-2_P1.3mm_Bridged2Bar_RoundedPad1.0x1.5mm, F.Cu at (141.8, 87.2)
- added Q10: AO3401A, Package_TO_SOT_SMD:SOT-23, F.Cu at (162.5, 66.2)
- C2, C59: value 100n -> 10u/50V; footprint Capacitor_SMD:C_0603_1608Metric -> Capacitor_SMD:C_1206_3216Metric
- C54, C8: value 220u/10V -> 100u / 6.3V; footprint Capacitor_THT:CP_Radial_D10.0mm_P2.50mm_P5.00mm -> Capacitor_SMD:C_1206_3216Metric
- C61: value 2.2u/25V -> 10u/50V; footprint Capacitor_SMD:C_0805_2012Metric -> Capacitor_SMD:C_1206_3216Metric
- C82: value 100u -> 100u / 6.3V
- L11: footprint Inductor_SMD:L_SXN_SMDRI74 -> Inductor_SMD:L_7.3x7.3_H4.5
- moved C82 124.8 mm to (150.8, 88.5), turned to 180 degrees
- moved C61 61.2 mm to (147.5, 100.7), turned to 90 degrees
- moved C59 57.1 mm to (149.5, 92.3), turned to -90 degrees
- moved C60 47.7 mm to (152.0, 92.3), turned to 90 degrees
- moved C45 46.9 mm to (150.2, 100.7), turned to 90 degrees
- moved FB1 46.3 mm to (144.0, 87.1), turned to 90 degrees
- moved C58 42.4 mm to (152.5, 101.2), turned to 90 degrees
- moved R14 40.5 mm to (141.0, 95.9), turned to -90 degrees
- moved C51 38.8 mm to (142.8, 94.5), turned to -90 degrees
- moved R13 37.4 mm to (144.2, 94.5), turned to -90 degrees
- moved Q7 37.3 mm to (159.1, 39.5), turned to -90 degrees
- moved C50 37.1 mm to (141.0, 92.7), turned to -90 degrees
- moved C6 36.8 mm to (156.0, 101.2), turned to 0 degrees
- moved C4 35.4 mm to (142.8, 91.0), turned to -90 degrees
- moved R12 33.8 mm to (144.2, 90.9), turned to -90 degrees
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Connections:
- net Net-(D2-K) renamed /Power/PH
- C11 pad 1: Net-(U1-DAC_OUTB) -> Net-(JP11-A)
- C2 pad 1: +3.3V -> GND
- C2 pad 2: GND -> Net-(U5-VIN)
- C54 pad 1: +3.3V -> GND
- C54 pad 2: GND -> +3.3V
- C59 pad 1: unconnected-(C59-Pad1) -> +3.3V
- C59 pad 2: unconnected-(C59-Pad2) -> GND
- C60 pad 1: unconnected-(C60-Pad1) -> GND
- C60 pad 2: unconnected-(C60-Pad2) -> +3.3V
- C61 pad 1: unconnected-(C61-Pad1) -> Net-(U5-VIN)
- C61 pad 2: unconnected-(C61-Pad2) -> GND
- C8 pad 1: +3.3V -> GND
- C8 pad 2: GND -> +3.3V
- C82 pad 1: unconnected-(C82-Pad1) -> +3.3V
- C82 pad 2: unconnected-(C82-Pad2) -> GND
- FB1 pad 1: unconnected-(FB1-Pad1) -> GND
- FB1 pad 2: unconnected-(FB1-Pad2) -> PGND
- JP5 pad 1: VIN -> Net-(JP5-A)
- Q3 pad 1: Net-(Q3-G) -> Net-(Q1-C)
- Q3 pad 2: Net-(JP3-B) -> VIN
- Q3 pad 3: Net-(J6-Pin_2) -> Net-(JP4-B)
- Q7 pad 1: Net-(D3-K) -> Net-(Q7-G)
- Q7 pad 2: Net-(JP5-B) -> Net-(JP3-B)
- Q7 pad 3: VIN -> Net-(J6-Pin_2)
- Q8 pad 1: Net-(Q3-G) -> Net-(Q7-G)
- Q9 pad 2: Net-(JP4-B) -> VIN
- Q9 pad 3: VIN -> Net-(JP4-B)
- R17 pad 2: Net-(Q3-G) -> Net-(Q7-G)
- R18 pad 1: VIN -> Net-(JP5-A)
- R21 pad 1: Net-(U1-DAC_OUTB) -> Net-(JP11-B)
- R5 pad 1: Net-(Q3-G) -> Net-(Q7-G)
- U1 pad 36: Net-(U1-DAC_OUTB) -> Net-(JP11-A)
Routing:
- net Net-(U5-VSENSE): track 0.00 -> 8.95 mm
- net Net-(U5-BOOT): track 0.00 -> 2.29 mm
- added copper zone on F.Cu, net +3.3V
- added copper zone on F.Cu, net /Power/PH
- added copper zone on B.Cu, net GND
- added copper zone on F.Cu, net GND

Commit message: Update SqueezeAMPagain.kicad_pcb, SqueezeAMPagain.kicad_prl, SqueezeAMPagain.kicad_pro, and 6 more files
Parts:
- added J11: Conn_02x06_Odd_Even, Connector_IDC:IDC-Header_2x06_P2.54mm_Vertical, F.Cu at (158.5, 55.0)
- L8, L9: value 4.7uH/3.0A -> 4.7uH/4.0A
- moved R19 22.3 mm to (138.5, 75.2)
- moved D3 18.5 mm to (142.0, 74.7), turned to -90 degrees
- moved Q6 18.4 mm to (145.0, 78.4)
- moved D4 18.3 mm to (78.7, 29.0)
- moved R16 18.2 mm to (143.7, 82.0), turned to 0 degrees
- moved R15 18.0 mm to (141.0, 81.8)
- moved JP4 17.7 mm to (143.5, 52.4), turned to 90 degrees
- moved Q10 16.8 mm to (146.6, 71.6)
- moved R18 16.5 mm to (146.7, 75.0)
- moved JP5 16.2 mm to (147.2, 68.0)
- moved C38 15.7 mm to (157.5, 41.0)
- moved FB5 14.8 mm to (148.0, 80.1), turned to -90 degrees
- moved C42 13.6 mm to (155.0, 39.8)
- moved NT2 12.3 mm to (155.0, 50.5), turned to -90 degrees
- moved C77 12.1 mm to (73.8, 31.2)
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Connections:
- net Net-(J6-Pin_2) renamed /Power/V_{supply}
- net VIN renamed V_{IN}
- C79 pad 2: unconnected-(C79-Pad2) -> GND
- C80 pad 2: unconnected-(C80-Pad2) -> GND
Routing:
- net +3.3V: track 0.00 -> 84.9 mm, vias 0 -> 4
- net /Amp/~{SPK_FAULT}: track 0.00 -> 49.0 mm, vias 0 -> 1
- net GND: track 17.4 -> 42.3 mm, vias 0 -> 4
- net Net-(U5-VIN): track 0.00 -> 23.4 mm, vias 0 -> 2
- net Net-(JP6-A): track 0.00 -> 17.0 mm
- net Net-(JP11-A): track 0.04 -> 15.8 mm
- net Net-(JP7-A): track 0.00 -> 13.4 mm
- net Net-(U5-VSENSE): track 8.95 -> 17.8 mm
- net Net-(U1-CP): track 0.89 -> 9.74 mm
- net PGND: track 2.42 -> 11.0 mm, vias 35 -> 36
- net Net-(U1-CN): track 0.00 -> 6.62 mm
- net Net-(U1-DVDD_REG): track 0.00 -> 5.02 mm
- net /Amp/SpeakerChannelB-/Cboot: track 0.00 -> 2.91 mm
- net Net-(C50-Pad2): track 0.00 -> 1.62 mm
- net /Amp/SpeakerChannelB+/Cboot: track 4.89 -> 6.28 mm
