File: SqueezeAMPagain/SqueezeAMPagain.kicad_pcb (KiCad board)
At the start: 2 copper layers, 109.5 x 108 mm, 176 parts, among them J1 Conn_01x02_Pin, J11 Conn_02x06_Odd_Even, J2 Conn_01x02_Pin, J3 Raspberry_Pi_2_3, J4 Conn_01x06_Pin, J5 USB_B_Micro, J6 Conn_01x02_Pin, J7 Barrel_Jack_Switch_MountingPin, J8 Conn_02x08_Odd_Even, J9 Conn_01x06_Pin, Q1 Q_NPN_BEC, Q10 AO3401A, Q3 AO3401A, Q4 Q_NPN_BEC, Q5 Q_NPN_BEC, Q6 Q_NPN_BEC, Q7 AO3401A, Q8 AO3401A, Q9 AO3401A, U1 TAS5756M, U2 RaspberryPi_Pico_W, U3 CP2102N-Axx-xQFN28, U4 ESP32-WROVER-E, U5 TPS5430DDA, U6 TSOP21xx, U7 AMS1117-3.3

Commit message: Update SqueezeAMPagain.kicad_pcb, SqueezeAMPagain.kicad_prl, SqueezeAMPagain.kicad_pro, and 7 more files
Parts:
- removed J11: Conn_02x06_Odd_Even, Connector_IDC:IDC-Header_2x06_P2.54mm_Vertical
- added C71: 100n, Capacitor_SMD:C_0603_1608Metric, F.Cu at (128.5, 101.3)
- added C81: 100n, Capacitor_SMD:C_0603_1608Metric, F.Cu at (139.5, 97.2)
- added FB2: 600Ω@100MHz 500mA, Inductor_SMD:L_0805_2012Metric, F.Cu at (134.0, 93.4)
- added J10: Conn_02x07_Odd_Even, Connector_IDC:IDC-Header_2x07_P2.54mm_Vertical, F.Cu at (157.0, 59.3)
- C54, C8, C82, C83: value 100u / 6.3V -> 47uF / 10V
- C59, C60: value 10u/50V -> 47uF / 10V
- C76: value 100n -> 2.2u/25V; footprint Capacitor_SMD:C_0603_1608Metric -> Capacitor_SMD:C_0805_2012Metric
- L11: footprint Inductor_SMD:L_7.3x7.3_H4.5 -> Inductor:L_Vishay_IHLP-3232
- R12: value 22k -> 15k
- R13: value 13k -> 4.7k
- moved U7 90.0 mm to (133.7, 99.5), turned to 180 degrees
- moved C76 80.8 mm to (131.5, 94.0), turned to -90 degrees
- moved R6 47.6 mm to (99.5, 82.7)
- moved R7 42.9 mm to (97.0, 82.7)
- moved Q4 41.7 mm to (96.9, 80.0)
- moved Q5 40.7 mm to (100.9, 80.5)
- moved C46 17.0 mm to (78.2, 51.5)
- moved C79 17.0 mm to (76.3, 41.5)
- moved C80 17.0 mm to (75.5, 45.5)
- moved R2 16.6 mm to (147.5, 63.5), turned to -90 degrees
- moved FB5 11.6 mm to (137.5, 85.0)
- moved R4 11.2 mm to (156.0, 49.5)
- moved R8 11.0 mm to (105.0, 80.0)
- moved JP4 10.5 mm to (150.7, 60.0), turned to 0 degrees
- moved U4 7.83 mm to (105.2, 103.7)
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Connections:
- C4 pad 1: +3.3V -> +5V
- C54 pad 2: +3.3V -> +5V
- C56 pad 1: +3.3V -> +5V
- C57 pad 1: +3.3V -> +5V
- C59 pad 1: +3.3V -> +5V
- C60 pad 2: +3.3V -> +5V
- C76 pad 1: +3.3V -> Net-(U7-VI)
- C8 pad 2: +3.3V -> +5V
- C82 pad 1: +3.3V -> +5V
- C83 pad 1: +3.3V -> +5V
- D3 pad 2: /Power/~{WAKE_DETECT} -> /Pico/GPIO6
- J3 pad 12: /Pi/BCLK -> /Amp/SCLK
- J3 pad 3: /Pi/SDA -> /SDA
- J3 pad 35: /Pi/LRCLK -> /Amp/LRCLK/FS
- J3 pad 40: /Pi/DATA -> /Amp/SDIN
- J3 pad 5: /Pi/SCL -> /SCL
- L11 pad 2: +3.3V -> +5V
- R12 pad 1: +3.3V -> +5V
- R2 pad 1: /Power/PON -> /Pico/GPIO7
- R20 pad 2: /Power/~{WAKE_DETECT} -> /Pico/GPIO6
- R26 pad 1: /Power/~{WAKE_DETECT} -> /Pico/GPIO6
- U2 pad 10: unconnected-(U2-GPIO7-Pad10) -> /Pico/GPIO7
- U2 pad 11: unconnected-(U2-GPIO8-Pad11) -> /esp/TCK
- U2 pad 12: unconnected-(U2-GPIO9-Pad12) -> /FPConnector/IO4
- U2 pad 13: Net-(U2-GND-Pad13) -> GND
- U2 pad 14: unconnected-(U2-GPIO10-Pad14) -> /FPConnector/IO3
- U2 pad 15: unconnected-(U2-GPIO11-Pad15) -> /FPConnector/IO2
- U2 pad 18: Net-(U2-GND-Pad13) -> GND
- U2 pad 21: unconnected-(U2-GPIO16-Pad21) -> /SDA
- U2 pad 22: unconnected-(U2-GPIO17-Pad22) -> /SCL
- U2 pad 23: Net-(U2-GND-Pad13) -> GND
- U2 pad 24: unconnected-(U2-GPIO18-Pad24) -> /FPConnector/IO1
- U2 pad 25: unconnected-(U2-GPIO19-Pad25) -> /esp/TDI
- U2 pad 26: unconnected-(U2-GPIO20-Pad26) -> /FPConnector/RESET
- U2 pad 28: Net-(U2-GND-Pad13) -> GND
- U2 pad 3: Net-(U2-GND-Pad13) -> GND
- U2 pad 38: Net-(U2-GND-Pad13) -> GND
- U2 pad 8: Net-(U2-GND-Pad13) -> GND
- U2 pad 9: unconnected-(U2-GPIO6-Pad9) -> /Pico/GPIO6
- U4 pad 12: /Power/PON -> /Pico/GPIO7
- U7 pad 3: V_{USB} -> Net-(U7-VI)
Routing:
- net +3.3V: track 84.9 -> 40.8 mm
- net +5V: track 0.00 -> 12.6 mm
Other:
- board size 109.5 x 108 mm -> 100.5 x 104 mm

Commit message: Update L_Radial_D12.0mm_P5+6+7.00mm_Fastron_11P.kicad_mod, SqueezeAMPagain.kicad_pcb, SqueezeAMPagain.kicad_prl, and 5 more files
Parts:
- removed FB3: 600Ω@100MHz 500mA, Inductor_SMD:L_0805_2012Metric
- added C84: 10u/50V, Capacitor_SMD:C_1206_3216Metric, F.Cu at (91.8, 57.0)
- added C85: 100n, Capacitor_SMD:C_0603_1608Metric, F.Cu at (126.2, 64.2)
- added C86: 100n, Capacitor_SMD:C_0603_1608Metric, F.Cu at (126.0, 58.3)
- added C87: 100n, Capacitor_SMD:C_0603_1608Metric, F.Cu at (98.8, 58.0)
- added C88: 100n, Capacitor_SMD:C_0603_1608Metric, F.Cu at (98.8, 64.0)
- moved R10 31.9 mm to (117.0, 105.6), turned to 180 degrees
- moved R1 31.5 mm to (100.5, 79.3), turned to -90 degrees
- moved R9 31.5 mm to (116.7, 103.3), turned to 180 degrees
- moved R11 26.9 mm to (117.0, 99.4), turned to 180 degrees
- moved R22 25.1 mm to (116.8, 104.4), turned to 180 degrees
- moved R23 24.0 mm to (116.7, 102.0), turned to 180 degrees
- moved R24 21.4 mm to (116.7, 100.4), turned to 0 degrees
- moved FB7 19.7 mm to (150.7, 75.4)
- moved R3 17.3 mm to (160.6, 52.9)
- moved Q1 16.9 mm to (160.7, 50.1)
- moved R2 15.1 mm to (156.9, 51.6)
- moved JP12 15.1 mm to (137.2, 72.8)
- moved FB1 14.5 mm to (139.5, 73.3)
- moved C44 10.9 mm to (135.6, 69.6), turned to -90 degrees
- moved Q10 9.76 mm to (144.7, 78.7), turned to -90 degrees
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Connections:
- net Net-(JP4-B) renamed /Power/V_{IN,SW}
- net Net-(Q1-E) renamed /Power/GND_{IN}
- C10 pad 2: GND -> PGND
- C12 pad 2: GND -> PGND
- C14 pad 2: GND -> PGND
- C16 pad 2: GND -> PGND
- C17 pad 2: GND -> PGND
- C18 pad 2: GNDA -> PGND
- C32 pad 2: GNDA -> PGND
- C33 pad 2: GND -> PGND
- C34 pad 2: GND -> PGND
- C35 pad 2: GND -> PGND
- C36 pad 2: GND -> PGND
- C37 pad 2: GND -> PGND
- J3 pad 19: unconnected-(J3-MOSI0/GPIO10-Pad19) -> /FPConnector/MOSI
- J3 pad 21: unconnected-(J3-MISO0/GPIO9-Pad21) -> /FPConnector/MISO
- J3 pad 22: unconnected-(J3-GPIO25-Pad22) -> /FPConnector/D/C
- J3 pad 23: unconnected-(J3-SCLK0/GPIO11-Pad23) -> /FPConnector/SCK
- J3 pad 24: unconnected-(J3-~{CE0}/GPIO8-Pad24) -> /FPConnector/CS
- JP6 pad 2: GND -> PGND
- JP7 pad 2: GND -> PGND
- R21 pad 2: GND -> PGND
- U1 pad 10: GNDA -> PGND
- U1 pad 15: GNDA -> PGND
- U1 pad 20: GND -> PGND
- U1 pad 26: GND -> PGND
- U1 pad 29: GND -> PGND
- U1 pad 33: GND -> PGND
Routing:
- net +3.3V: track 40.8 -> 249.7 mm, vias 4 -> 7
- net /SDA: track 37.7 -> 206.8 mm, vias 0 -> 5
- net /SCL: track 41.0 -> 170.2 mm, vias 0 -> 6
- net /Pico/GPIO7: track 0.00 -> 125.2 mm, vias 0 -> 3
- net /FPConnector/SCK: track 0.00 -> 123.7 mm, vias 0 -> 3
- net /esp/TCK: track 0.00 -> 118.3 mm, vias 0 -> 2
- net /FPConnector/IO3: track 0.00 -> 102.2 mm, vias 0 -> 3
- net /FPConnector/MISO: track 0.00 -> 101.5 mm, vias 0 -> 4
- net /FPConnector/D/C: track 0.00 -> 93.8 mm, vias 0 -> 3
- net /FPConnector/IO4: track 0.00 -> 93.1 mm, vias 0 -> 1
- net /USB-Uart/TX: track 0.00 -> 91.3 mm, vias 0 -> 1
- net /USB-Uart/EN/~{RESET}: track 0.00 -> 90.9 mm, vias 0 -> 3
- net /FPConnector/IO2: track 0.00 -> 90.4 mm, vias 0 -> 2
- net +5V: track 12.6 -> 93.9 mm, vias 0 -> 1
- net /FPConnector/CS: track 0.00 -> 76.9 mm, vias 0 -> 2
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- added copper zone on F.Cu, net +5V
- added copper zone on B.Cu, net /Power/GND_{IN}
- added copper zone on F.Cu, net /Power/V_{IN,SW}
- added copper zone on F.Cu, net V_{IN}
- removed copper zone on F.Cu, net +3.3V
- removed copper zone on B.Cu, net /Amp/SPK_B+
