File: SqueezeAMPagain/pico.kicad_sch (KiCad schematic)
At the start: 1 part, among them U2 RaspberryPi_Pico_W

Commit message: Update .gitignore, L_Radial_D12.0mm_P5+6+7.00mm_Fastron_11P.kicad_mod, SqueezeAMPagain.kicad_pcb, and 13 more files
Parts:
- added C53, C55: 100n, Capacitor_SMD:C_0603_1608Metric, symbol Device:C
Connections:
- net TX: now reaches U2.1 (GPIO0)
- net MCLK: now reaches U2.16 (GPIO12)
- net BCLK: now reaches U2.19 (GPIO14)
- net RX: now reaches U2.2 (GPIO1)
- net DATA: now reaches U2.20 (GPIO15)
- net SPI0_SCK: now reaches U2.4 (GPIO2)
- net SPI0_MOSI: now reaches U2.5 (GPIO3)
- net SPI0_MISO: now reaches U2.6 (GPIO4)
- net SPI0_CS: now reaches U2.7 (GPIO5)
- new net +3.3V: C53.1, C55.1
- new net GND: C53.2, C55.2

Commit message: Update SqueezeAMPagain.kicad_pcb, SqueezeAMPagain.kicad_prl, USB-Uart.kicad_sch, and 4 more files
Parts:
- added R10, R11, R8, R9: 33, Resistor_SMD:R_0402_1005Metric, symbol Device:R
Connections:
- net BCLK: now also R9.1; no longer U2.19 (GPIO14)
- net DATA: now also R10.1; no longer U2.20 (GPIO15)
- net LRCLK: now also R11.1
- net MCLK: now also R8.1; no longer U2.16 (GPIO12)
- net at U2.17 (GPIO13): now also R11.2
- new net: R8.2, U2.16 (GPIO12)
- new net: R10.2, U2.20 (GPIO15)
- new net: R9.2, U2.19 (GPIO14)

Commit message: Update SqueezeAMPagain.kicad_pcb, SqueezeAMPagain.kicad_prl, SqueezeAMPagain.kicad_pro, and 7 more files
Connections:
- net GND: now also U2.13 (GND), U2.18 (GND), U2.23 (GND), U2.28 (GND), U2.3 (GND), U2.38 (GND), U2.8 (GND)
- net SCL: now also U2.22 (GPIO17)
- net SDA: now also U2.21 (GPIO16)
- net GPIO7: now reaches U2.10 (GPIO7)
- net GPIO8: now reaches U2.11 (GPIO8)
- net GPIO9: now reaches U2.12 (GPIO9)
- net GPIO10: now reaches U2.14 (GPIO10)
- net GPIO11: now reaches U2.15 (GPIO11)
- net GPIO18: now reaches U2.24 (GPIO18)
- net GPIO19: now reaches U2.25 (GPIO19)
- net GPIO20: now reaches U2.26 (GPIO20)
- net GPIO6: now reaches U2.9 (GPIO6)
Changed lines of the file:
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@@
+		)
+	)
+	(hierarchical_label "GPIO9"
+		(shape bidirectional)
+		(at 104.14 93.98 180)
+		(fields_autoplaced yes)
+		(effects
+			(font
+				(size 1.27 1.27)
+			)
+			(justify right)
 		)
 	)
@@
 	(hierarchical_label "SCL"
 		(shape output)
-		(at 191.77 124.46 0)
+		(at 149.86 81.28 0)
 		(fields_autoplaced yes)
 		(effects
@@
 		)
 	)
+	(hierarchical_label "GPIO19"
+		(shape bidirectional)
+		(at 149.86 86.36 0)
+		(fields_autoplaced yes)
+		(effects
+			(font
+				(size 1.27 1.27)
+			)
+			(justify left)
+		)
+	)
+	(hierarchical_label "GPIO20"
+		(shape bidirectional)
+		(at 149.86 88.9 0)
+		(fields_autoplaced yes)
+		(effects
+			(font
+				(size 1.27 1.27)
+			)
+			(justify left)
+		)
+	)
 	(hierarchical_label "SDA"
 		(shape bidirectional)
-		(at 191.77 121.92 0)
+		(at 149.86 78.74 0)
 		(fields_autoplaced yes)
 		(effects
@@
 			)
 			(justify left)
+		)
+	)
+	(hierarchical_label "GPIO7"
+		(shape bidirectional)
+		(at 104.14 88.9 180)
+		(fields_autoplaced yes)
+		(effects
+			(font
+				(size 1.27 1.27)
+			)
+			(justify right)
 		)
 	)
@@
 		)
 	)
+	(hierarchical_label "GPIO6"
+		(shape bidirectional)
+		(at 104.14 86.36 180)
+		(fields_autoplaced yes)
+		(effects
+			(font
+				(size 1.27 1.27)
+			)
+			(justify right)
+		)
+	)
+	(hierarchical_label "GPIO11"
+		(shape bidirectional)
+		(at 104.14 99.06 180)
+		(fields_autoplaced yes)
+		(effects
+			(font
+				(size 1.27 1.27)
+			)
+			(justify right)
+		)
+	)
 	(hierarchical_label "TX"
 		(shape output)
@@
 		)
 	)
+	(hierarchical_label "GPIO18"
+		(shape bidirectional)
+		(at 149.86 83.82 0)
+		(fields_autoplaced yes)
+		(effects
+			(font
+				(size 1.27 1.27)
+			)
+			(justify left)
+		)
+	)
 	(hierarchical_label "BCLK"
 		(shape output)
@@
 		(shape output)
 		(at 91.44 83.82 180)
+		(fields_autoplaced yes)
+		(effects
+			(font
+				(size 1.27 1.27)
+			)
+			(justify right)
+		)
+	)
+	(hierarchical_label "GPIO8"
+		(shape bidirectional)
+		(at 104.14 91.44 180)
+		(fields_autoplaced yes)
+		(effects
+			(font
+				(size 1.27 1.27)
+			)
+			(justify right)
+		)
+	)
+	(hierarchical_label "GPIO10"
+		(shape bidirectional)
+		(at 104.14 96.52 180)
 		(fields_autoplaced yes)
 		(effects
@@
 					(unit 1)
 				)
+			)
+		)
+	)
+	(symbol
+		(lib_id "power:GND")
+		(at 127 132.08 0)
+		(unit 1)
+		(exclude_from_sim no)
+		(in_bom yes)
+		(on_board yes)
+		(dnp no)
+		(fields_autoplaced yes)
+		(property "Reference" "#PWR0119"
+			(at 127 138.43 0)
+			(effects
+				(font
+					(size 1.27 1.27)
+				)
+				(hide yes)
+			)
+		)
+		(property "Value" "GND"
+			(at 127 137.16 0)
+			(effects
+				(font
+					(size 1.27 1.27)
+				)
+			)
+		)
+		(property "Footprint" ""
+			(at 127 132.08 0)
+			(effects
+				(font
+					(size 1.27 1.27)
+				)
+				(hide yes)
+			)
+		)
+		(property "Datasheet" ""
+			(at 127 132.08 0)
+			(effects
+				(font
+					(size 1.27 1.27)
+				)
+				(hide yes)
+			)
+		)
+		(property "Description" "Power symbol creates a global label with name \"GND\" , ground"
+			(at 127 132.08 0)
+			(effects
+				(font
+					(size 1.27 1.27)
+				)
+				(hide yes)
+			)
+		)
+		(pin "1"
+		)
+		(instances
+			(project "SqueezeAMPagain"
+				(path "/3675160b-d9e5-490e-b506-2a7966e79ed0/e8aa0c29-7d4a-4486-816f-de6795c685f9"
+					(reference "#PWR0119")
+					(unit 1)
+				)

Commit message: Update SqueezeAMPagain.kicad_pcb, SqueezeAMPagain.kicad_prl, SqueezeAMPagain.kicad_pro, and 5 more files
Parts:
- added C89, C90: 100n, Capacitor_SMD:C_0603_1608Metric, symbol Device:C
- added JP13: LV On, Jumper:SolderJumper-2_P1.3mm_Open_RoundedPad1.0x1.5mm, symbol Jumper:SolderJumper_2_Open
- U2: footprint pipico:RaspberryPi_Pico_Common_THT -> pipico_reduced:RaspberryPi_Pico_Common_THT_nokeepout
Connections:
- net +3.3V: now also JP13.2 (B)
- net GND: now also C89.2, C90.2
- net GPIO18: now also U2.4 (GPIO2); no longer U2.24 (GPIO18)
- net GPIO19: now also U2.5 (GPIO3); no longer U2.25 (GPIO19)
- net GPIO20: now also U2.6 (GPIO4); no longer U2.26 (GPIO20)
- net SCL: now also U2.27 (GPIO21); no longer U2.22 (GPIO17)
- net SDA: now also U2.26 (GPIO20); no longer U2.21 (GPIO16)
- net SPI0_CS: now also U2.22 (GPIO17); no longer U2.7 (GPIO5)
- net SPI0_MISO: now also U2.21 (GPIO16); no longer U2.6 (GPIO4)
- net SPI0_MOSI: now also U2.25 (GPIO19); no longer U2.5 (GPIO3)
- net SPI0_SCK: now also U2.24 (GPIO18); no longer U2.4 (GPIO2)
- net GPIO29: now reaches U2.29 (GPIO22)
- net at U2.36 (3V3): now also C89.1, JP13.1 (A)
- net +5V: now reaches U2.39 (VSYS)
- net +5V: now also C90.1
Other:
- moved on the sheet: C53, C55

Commit message: Update SqueezeAMPagain.kicad_pcb, SqueezeAMPagain.kicad_prl, SqueezeAMPagain.kicad_pro, and 5 more files
Parts:
- removed C53: 100n, Capacitor_SMD:C_0603_1608Metric, symbol Device:C
Changed lines of the file:
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@@
-	)
-	(symbol
-		(lib_id "Device:C")
-		(at 82.55 26.67 0)
-		(unit 1)
-		(exclude_from_sim no)
-		(in_bom yes)
-		(on_board yes)
-		(dnp no)
-		(fields_autoplaced yes)
-		(property "Reference" "C53"
-			(at 86.36 25.3999 0)
-			(effects
-				(font
-					(size 1.27 1.27)
-				)
-				(justify left)
-			)
-		)
-		(property "Value" "100n"
-			(at 86.36 27.9399 0)
-			(effects
-				(font
-					(size 1.27 1.27)
-				)
-				(justify left)
-			)
-		)
-		(property "Footprint" "Capacitor_SMD:C_0603_1608Metric"
-			(at 83.5152 30.48 0)
-			(effects
-				(font
-					(size 1.27 1.27)
-				)
-				(hide yes)
-			)
-		)
-		(property "Datasheet" "~"
-			(at 82.55 26.67 0)
-			(effects
-				(font
-					(size 1.27 1.27)
-				)
-				(hide yes)
-			)
-		)
-		(property "Description" "Unpolarized capacitor"
-			(at 82.55 26.67 0)
-			(effects
-				(font
-					(size 1.27 1.27)
-				)
-				(hide yes)
-			)
-		)
-		(pin "2"
-		)
-		(pin "1"
-		)
-		(instances
-			(project "SqueezeAMPagain"
-				(path "/3675160b-d9e5-490e-b506-2a7966e79ed0/e8aa0c29-7d4a-4486-816f-de6795c685f9"
-					(reference "C53")
-					(unit 1)
-				)
-			)
-		)
 	)
 	(symbol
@@
 	)
 	(symbol
-		(lib_id "power:GND")
-		(at 82.55 30.48 0)
-		(unit 1)
-		(exclude_from_sim no)
-		(in_bom yes)
-		(on_board yes)
-		(dnp no)
-		(fields_autoplaced yes)
-		(property "Reference" "#PWR077"
-			(at 82.55 36.83 0)
-			(effects
-				(font
-					(size 1.27 1.27)
-				)
-				(hide yes)
-			)
-		)
-		(property "Value" "GND"
-			(at 82.55 35.56 0)
-			(effects
-				(font
-					(size 1.27 1.27)
-				)
-			)
-		)
-		(property "Footprint" ""
-			(at 82.55 30.48 0)
-			(effects
-				(font
-					(size 1.27 1.27)
-				)
-				(hide yes)
-			)
-		)
-		(property "Datasheet" ""
-			(at 82.55 30.48 0)
-			(effects
-				(font
-					(size 1.27 1.27)
-				)
-				(hide yes)
-			)
-		)
-		(property "Description" "Power symbol creates a global label with name \"GND\" , ground"
-			(at 82.55 30.48 0)
-			(effects
-				(font
-					(size 1.27 1.27)
-				)
-				(hide yes)
-			)
-		)
-		(pin "1"
-		)
-		(instances
-			(project "SqueezeAMPagain"
-				(path "/3675160b-d9e5-490e-b506-2a7966e79ed0/e8aa0c29-7d4a-4486-816f-de6795c685f9"
-					(reference "#PWR077")
-					(unit 1)
-				)
-			)
-		)
-	)
-	(symbol
 		(lib_id "Device:C")
 		(at 97.79 26.67 0)
@@
 					(unit 1)
 				)
-			)
-		)
-	)
-	(symbol
-		(lib_id "power:+3.3V")
-		(at 82.55 22.86 0)
-		(unit 1)
-		(exclude_from_sim no)
-		(in_bom yes)
-		(on_board yes)
-		(dnp no)
-		(fields_autoplaced yes)
-		(property "Reference" "#PWR076"
-			(at 82.55 26.67 0)
-			(effects
-				(font
-					(size 1.27 1.27)
-				)
-				(hide yes)
-			)
-		)
-		(property "Value" "+3.3V"
-			(at 82.55 17.78 0)
-			(effects
-				(font
-					(size 1.27 1.27)
-				)
-			)
-		)
-		(property "Footprint" ""
-			(at 82.55 22.86 0)
-			(effects
-				(font
-					(size 1.27 1.27)
-				)
-				(hide yes)
-			)
-		)
-		(property "Datasheet" ""
-			(at 82.55 22.86 0)
-			(effects
-				(font
-					(size 1.27 1.27)
-				)
-				(hide yes)
-			)
-		)
-		(property "Description" "Power symbol creates a global label with name \"+3.3V\""
-			(at 82.55 22.86 0)
-			(effects
-				(font
-					(size 1.27 1.27)
-				)
-				(hide yes)
-			)
-		)
-		(pin "1"
-		)
-		(instances
-			(project "SqueezeAMPagain"
-				(path "/3675160b-d9e5-490e-b506-2a7966e79ed0/e8aa0c29-7d4a-4486-816f-de6795c685f9"
-					(reference "#PWR076")
-					(unit 1)
-				)

Commit message: Update SqueezeAMPagain.kicad_pcb, SqueezeAMPagain.kicad_prl, SqueezeAMPagain.kicad_pro, and 11 more files
Parts:
- renumbered C55 to C56, C89 to C57, C90 to C58, JP13 to JP9, R8 to R18, R11 to R19, R9 to R20, R10 to R21, U2 to U3
Changed lines of the file:
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@@
 		(dnp no)
 		(fields_autoplaced yes)
-		(property "Reference" "C90"
+		(property "Reference" "C58"
 			(at 163.83 46.9899 0)
 			(effects
@@
 			(project "SqueezeAMPagain"
 				(path "/3675160b-d9e5-490e-b506-2a7966e79ed0/e8aa0c29-7d4a-4486-816f-de6795c685f9"
-					(reference "C90")
+					(reference "C58")
 					(unit 1)
 				)
@@
 		(dnp no)
 		(fields_autoplaced yes)
-		(property "Reference" "#PWR053"
+		(property "Reference" "#PWR073"
 			(at 160.02 58.42 0)
 			(effects
@@
 			(project "SqueezeAMPagain"
 				(path "/3675160b-d9e5-490e-b506-2a7966e79ed0/e8aa0c29-7d4a-4486-816f-de6795c685f9"
-					(reference "#PWR053")
+					(reference "#PWR073")
 					(unit 1)
 				)
@@
 		(dnp no)
 		(fields_autoplaced yes)
-		(property "Reference" "R11"
+		(property "Reference" "R19"
 			(at 67.31 97.79 90)
 			(effects
@@
 			(project "SqueezeAMPagain"
 				(path "/3675160b-d9e5-490e-b506-2a7966e79ed0/e8aa0c29-7d4a-4486-816f-de6795c685f9"
-					(reference "R11")
+					(reference "R19")
 					(unit 1)
 				)
@@
 		(dnp no)
 		(fields_autoplaced yes)
-		(property "Reference" "#PWR078"
+		(property "Reference" "#PWR066"
 			(at 97.79 26.67 0)
 			(effects
@@
 			(project "SqueezeAMPagain"
 				(path "/3675160b-d9e5-490e-b506-2a7966e79ed0/e8aa0c29-7d4a-4486-816f-de6795c685f9"
-					(reference "#PWR078")
+					(reference "#PWR066")
 					(unit 1)
 				)
@@
 		(dnp no)
 		(fields_autoplaced yes)
-		(property "Reference" "#PWR055"
+		(property "Reference" "#PWR072"
 			(at 160.02 48.26 0)
 			(effects
@@
 			(project "SqueezeAMPagain"
 				(path "/3675160b-d9e5-490e-b506-2a7966e79ed0/e8aa0c29-7d4a-4486-816f-de6795c685f9"
-					(reference "#PWR055")
+					(reference "#PWR072")
 					(unit 1)
 				)
@@
 		(dnp no)
 		(fields_autoplaced yes)
-		(property "Reference" "R8"
+		(property "Reference" "R18"
 			(at 58.42 95.25 90)
 			(effects
@@
 			(project "SqueezeAMPagain"
 				(path "/3675160b-d9e5-490e-b506-2a7966e79ed0/e8aa0c29-7d4a-4486-816f-de6795c685f9"
-					(reference "R8")
+					(reference "R18")
 					(unit 1)
 				)
@@
 		(dnp no)
 		(fields_autoplaced yes)
-		(property "Reference" "#PWR047"
+		(property "Reference" "#PWR068"
 			(at 113.03 55.88 0)
 			(effects
@@
 			(project "SqueezeAMPagain"
 				(path "/3675160b-d9e5-490e-b506-2a7966e79ed0/e8aa0c29-7d4a-4486-816f-de6795c685f9"
-					(reference "#PWR047")
+					(reference "#PWR068")
 					(unit 1)
 				)
@@
 		(dnp no)
 		(fields_autoplaced yes)
-		(property "Reference" "C89"
+		(property "Reference" "C57"
 			(at 116.84 44.4499 0)
 			(effects
@@
 			(project "SqueezeAMPagain"
 				(path "/3675160b-d9e5-490e-b506-2a7966e79ed0/e8aa0c29-7d4a-4486-816f-de6795c685f9"
-					(reference "C89")
+					(reference "C57")
 					(unit 1)
 				)
@@
 		(dnp no)
 		(fields_autoplaced yes)
-		(property "Reference" "R10"
+		(property "Reference" "R21"
 			(at 85.09 102.87 90)
 			(effects
@@
 			(project "SqueezeAMPagain"
 				(path "/3675160b-d9e5-490e-b506-2a7966e79ed0/e8aa0c29-7d4a-4486-816f-de6795c685f9"
-					(reference "R10")
+					(reference "R21")
 					(unit 1)
 				)
@@
 		(dnp no)
 		(fields_autoplaced yes)
-		(property "Reference" "C55"
+		(property "Reference" "C56"
 			(at 101.6 25.3999 0)
 			(effects
@@
 			(project "SqueezeAMPagain"
 				(path "/3675160b-d9e5-490e-b506-2a7966e79ed0/e8aa0c29-7d4a-4486-816f-de6795c685f9"
-					(reference "C55")
+					(reference "C56")
 					(unit 1)
 				)
@@
 		(dnp no)
 		(fields_autoplaced yes)
-		(property "Reference" "R9"
+		(property "Reference" "R20"
 			(at 76.2 100.33 90)
 			(effects
@@
 			(project "SqueezeAMPagain"
 				(path "/3675160b-d9e5-490e-b506-2a7966e79ed0/e8aa0c29-7d4a-4486-816f-de6795c685f9"
-					(reference "R9")
+					(reference "R20")
 					(unit 1)
 				)
@@
 		(dnp no)
 		(fields_autoplaced yes)
-		(property "Reference" "#PWR0119"
+		(property "Reference" "#PWR071"
 			(at 127 138.43 0)
 			(effects
@@
 			(project "SqueezeAMPagain"
 				(path "/3675160b-d9e5-490e-b506-2a7966e79ed0/e8aa0c29-7d4a-4486-816f-de6795c685f9"
-					(reference "#PWR0119")
+					(reference "#PWR071")
 					(unit 1)
 				)
@@
 		(dnp no)
 		(fields_autoplaced yes)
-		(property "Reference" "JP13"
+		(property "Reference" "JP9"
 			(at 124.46 33.0199 90)
 			(effects
@@
 			(project "SqueezeAMPagain"
 				(path "/3675160b-d9e5-490e-b506-2a7966e79ed0/e8aa0c29-7d4a-4486-816f-de6795c685f9"
-					(reference "JP13")
+					(reference "JP9")
 					(unit 1)
 				)
@@
 		(dnp no)
 		(fields_autoplaced yes)
-		(property "Reference" "#PWR079"
+		(property "Reference" "#PWR067"
 			(at 97.79 36.83 0)
 			(effects
@@
 			(project "SqueezeAMPagain"
 				(path "/3675160b-d9e5-490e-b506-2a7966e79ed0/e8aa0c29-7d4a-4486-816f-de6795c685f9"
-					(reference "#PWR079")
+					(reference "#PWR067")
 					(unit 1)
 				)
@@
 		(dnp no)
 		(fields_autoplaced yes)
-		(property "Reference" "U2"
+		(property "Reference" "U3"
 			(at 129.1941 130.81 0)
 			(effects
@@
 			(project "SqueezeAMPagain"
 				(path "/3675160b-d9e5-490e-b506-2a7966e79ed0/e8aa0c29-7d4a-4486-816f-de6795c685f9"
-					(reference "U2")
+					(reference "U3")
 					(unit 1)
 				)
@@
 		(dnp no)
 		(fields_autoplaced yes)
-		(property "Reference" "#PWR045"
+		(property "Reference" "#PWR070"
 			(at 127 50.8 0)
 			(effects
@@
 			(project "SqueezeAMPagain"
 				(path "/3675160b-d9e5-490e-b506-2a7966e79ed0/e8aa0c29-7d4a-4486-816f-de6795c685f9"
-					(reference "#PWR045")
+					(reference "#PWR070")
 					(unit 1)
 				)
@@
 		(dnp no)
 		(fields_autoplaced yes)
-		(property "Reference" "#PWR046"
+		(property "Reference" "#PWR069"
 			(at 121.92 34.29 0)
 			(effects
@@
 			(project "SqueezeAMPagain"
 				(path "/3675160b-d9e5-490e-b506-2a7966e79ed0/e8aa0c29-7d4a-4486-816f-de6795c685f9"
-					(reference "#PWR046")
-					(unit 1)
-				)
+					(reference "#PWR069")
+					(unit 1)
+				)

Commit message: Update SqueezeAMPagain.kicad_pcb, SqueezeAMPagain.kicad_prl, SqueezeAMPagain.kicad_pro, and 7 more files
Other:
- note added: ""P" for pico"
Changed lines of the file:
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@@
+		)
+	)
+	(polyline
+		(pts
+			(xy 55.88 116.84) (xy 64.77 116.84)
+		)
+		(stroke
+			(width 0)
+			(type default)
 		)
 	)
@@
 		)
 	)
+	(polyline
+		(pts
+			(xy 88.9 115.57) (xy 88.9 116.84)
+		)
+		(stroke
+			(width 0)
+			(type default)
+		)
+	)
 	(wire
 		(pts
@@
 		)
 	)
+	(polyline
+		(pts
+			(xy 55.88 115.57) (xy 55.88 116.84)
+		)
+		(stroke
+			(width 0)
+			(type default)
+		)
+	)
 	(wire
 		(pts
@@
 		)
 	)
+	(polyline
+		(pts
+			(xy 77.47 116.84) (xy 88.9 116.84)
+		)
+		(stroke
+			(width 0)
+			(type default)
+		)
+	)
 	(wire
 		(pts
@@
 		)
 	)
+	(text "\"P\" for pico"
+		(exclude_from_sim no)
+		(at 70.612 117.094 0)
+		(effects
+			(font
+				(size 1.27 1.27)
+			)
+		)
+	)

Commit message: Update SqueezeAMPagain.kicad_pcb, SqueezeAMPagain.kicad_prl, SqueezeAMPagain.kicad_pro, and 11 more files
Other:
- title: (none) -> SqueezeAMP_{again}
- moved on the sheet: C56
Changed lines of the file:
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@@
 	(generator_version "8.0")
 	(paper "A4")
+	(title_block
+		(title "SqueezeAMP_{again}")
+		(date "2024-08-23")
+		(rev "1.0")
+		(comment 1 "Raspberry Pi Pico W option")
+	)
 	(junction
 		(at 121.92 40.64)
@@
 	(symbol
 		(lib_id "power:+3.3V")
-		(at 97.79 22.86 0)
+		(at 173.99 44.45 0)
 		(unit 1)
 		(exclude_from_sim no)
@@
 		(fields_autoplaced yes)
 		(property "Reference" "#PWR066"
-			(at 97.79 26.67 0)
+			(at 173.99 48.26 0)
 			(effects
 				(font
@@
 		)
 		(property "Value" "+3.3V"
-			(at 97.79 17.78 0)
+			(at 173.99 39.37 0)
 			(effects
 				(font
@@
 		)
 		(property "Footprint" ""
-			(at 97.79 22.86 0)
+			(at 173.99 44.45 0)
 			(effects
 				(font
@@
 		)
 		(property "Datasheet" ""
-			(at 97.79 22.86 0)
+			(at 173.99 44.45 0)
 			(effects
 				(font
@@
 		)
 		(property "Description" "Power symbol creates a global label with name \"+3.3V\""
-			(at 97.79 22.86 0)
+			(at 173.99 44.45 0)
 			(effects
 				(font
@@
 	(symbol
 		(lib_id "Device:C")
-		(at 97.79 26.67 0)
+		(at 173.99 48.26 0)
 		(unit 1)
 		(exclude_from_sim no)
@@
 		(fields_autoplaced yes)
 		(property "Reference" "C56"
-			(at 101.6 25.3999 0)
+			(at 177.8 46.9899 0)
 			(effects
 				(font
@@
 		)
 		(property "Value" "100n"
-			(at 101.6 27.9399 0)
+			(at 177.8 49.5299 0)
 			(effects
 				(font
@@
 		)
 		(property "Footprint" "Capacitor_SMD:C_0603_1608Metric"
-			(at 98.7552 30.48 0)
+			(at 174.9552 52.07 0)
 			(effects
 				(font
@@
 		)
 		(property "Datasheet" "~"
-			(at 97.79 26.67 0)
+			(at 173.99 48.26 0)
 			(effects
 				(font
@@
 		)
 		(property "Description" "Unpolarized capacitor"
-			(at 97.79 26.67 0)
+			(at 173.99 48.26 0)
 			(effects
 				(font
@@
 	(symbol
 		(lib_id "power:GND")
-		(at 97.79 30.48 0)
+		(at 173.99 52.07 0)
 		(unit 1)
 		(exclude_from_sim no)
@@
 		(fields_autoplaced yes)
 		(property "Reference" "#PWR067"
-			(at 97.79 36.83 0)
+			(at 173.99 58.42 0)
 			(effects
 				(font
@@
 		)
 		(property "Value" "GND"
-			(at 97.79 35.56 0)
+			(at 173.99 57.15 0)
 			(effects
 				(font
@@
 		)
 		(property "Footprint" ""
-			(at 97.79 30.48 0)
+			(at 173.99 52.07 0)
 			(effects
 				(font
@@
 		)
 		(property "Datasheet" ""
-			(at 97.79 30.48 0)
+			(at 173.99 52.07 0)
 			(effects
 				(font
@@
 		)
 		(property "Description" "Power symbol creates a global label with name \"GND\" , ground"
-			(at 97.79 30.48 0)
-			(effects
-				(font
+			(at 173.99 52.07 0)
+			(effects
+				(font
