File: SqueezeAMPagain/spkchannel.kicad_sch (KiCad schematic)
At the start: 6 parts

Commit message: v2
Parts:
- L2: renamed from L11; value 4.7uH/6.0A -> 4.7uH
- renumbered C52 to C40, C53 to C41, C54 to C42, C55 to C43, L12 to L3
Changed lines of the file:
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@@
 (kicad_sch
-	(version 20231120)
+	(version 20250114)
 	(generator "eeschema")
-	(generator_version "8.0")
+	(generator_version "9.0")
 	(paper "A4")
 	(title_block
@@
 		(rev "1.0")
 	)
+	(text_box "\nSuitable inductors for more Power:\nd ≤ 12mm, Grid 5mm\n\n- WE 7447471047  <- shielded\n\n- Fastron 07HCP-4R7M-50 <- only 4A\n"
+		(exclude_from_sim yes)
+		(at 73.66 83.82 0)
+		(size 44.45 17.78)
+		(margins 0.9525 0.9525 0.9525 0.9525)
+		(stroke
+			(width 0)
+			(type solid)
+		)
+		(fill
+			(type none)
+		)
+		(effects
+			(font
+				(size 1.27 1.27)
+			)
+			(justify left top)
+		)
+	)
 	(junction
 		(at 163.83 85.09)
@@
 			(width 0)
 			(type default)
-		)
-	)
-	(text_box "Suitable inductors:\nd ≤ 12mm, Grid 5mm\n\n- WE 7447471047  <- shielded\n\n- Fastron 07HCP-4R7M-50 <- only 4A\n"
-		(exclude_from_sim yes)
-		(at 73.66 83.82 0)
-		(size 44.45 17.78)
-		(stroke
-			(width 0)
-			(type default)
-		)
-		(fill
-			(type none)
-		)
-		(effects
-			(font
-				(size 1.27 1.27)
-			)
-			(justify left top)
 		)
 	)
@@
 		(dnp no)
 		(fields_autoplaced yes)
-		(property "Reference" "C52"
+		(property "Reference" "C40"
 			(at 102.87 48.2599 0)
 			(effects
@@
 		(dnp no)
 		(fields_autoplaced yes)
-		(property "Reference" "C53"
+		(property "Reference" "C41"
 			(at 142.24 77.4699 0)
 			(effects
@@
 		(dnp yes)
 		(fields_autoplaced yes)
-		(property "Reference" "L12"
+		(property "Reference" "L3"
 			(at 113.03 71.12 90)
 			(effects
@@
 		(dnp no)
 		(fields_autoplaced yes)
-		(property "Reference" "L11"
+		(property "Reference" "L2"
 			(at 113.03 62.23 90)
 			(effects
@@
 			)
 		)
-		(property "Value" "4.7uH/6.0A"
+		(property "Value" "4.7uH"
 			(at 113.03 64.77 90)
 			(effects
@@
 		(dnp no)
 		(fields_autoplaced yes)
-		(property "Reference" "C54"
+		(property "Reference" "C42"
 			(at 156.21 77.4699 0)
 			(effects
@@
 		(dnp no)
 		(fields_autoplaced yes)
-		(property "Reference" "#PWR060"
+		(property "Reference" "#PWR057"
 			(at 163.83 95.25 0)
 			(effects
@@
 		(dnp no)
 		(fields_autoplaced yes)
-		(property "Reference" "C55"
+		(property "Reference" "C43"
 			(at 167.64 77.4699 0)
 			(effects
