File: SqueezeAMPagain/SqueezeAMPagain.kicad_sch (KiCad schematic)
At the start: 8 parts

Commit message: Update SqueezeAMPagain.kicad_pcb, SqueezeAMPagain.kicad_prl, SqueezeAMPagain.kicad_pro, and 5 more files
Parts:
- added H6: MountingHole, MountingHole:MountingHole_2.5mm, symbol Mechanical:MountingHole
- added TP1: 3V3, TestPoint:TestPoint_Pad_D1.0mm, symbol Connector:TestPoint
- added TP2: 3V3_{SW}, TestPoint:TestPoint_Pad_D1.0mm, symbol Connector:TestPoint
- added TP3: PVDD, TestPoint:TestPoint_Pad_D1.0mm, symbol Connector:TestPoint
- added TP4: V_{IN}, TestPoint:TestPoint_Pad_D1.0mm, symbol Connector:TestPoint
Connections:
- net +3.3V: now also TP1.1
- new net +3.3V_{SW}: TP2.1
- new net PVDD: TP3.1
- new net V_{IN}: TP4.1
Other:
- note added: "Heat spreader M2:"
- note added: "M3 x 4:"

Commit message: Update SqueezeAMPagain.kicad_pcb, SqueezeAMPagain.kicad_prl, SqueezeAMPagain.kicad_pro, and 7 more files
Parts:
- added TP10, TP11, TP6, TP7, TP8, TP9: ~, TestPoint:TestPoint_Pad_D1.0mm, symbol Connector:TestPoint
- added TP12: ~, TestPoint:TestPoint_THTPad_D1.0mm_Drill0.5mm, symbol Connector:TestPoint
- added TP5: Mclk, TestPoint:TestPoint_Pad_D1.0mm, symbol Connector:TestPoint
Connections:
- net Amp/LRCLK/FS: now also TP7.1
- net Amp/MCLK: now also TP5.1
- net Amp/SCLK: now also TP6.1
- net Amp/SDIN: now also TP8.1
- net SCL: now also TP9.1
- net SDA: now also TP10.1
- new net +5V: TP11.1
- new net GND: TP12.1

Commit message: Update SqueezeAMPagain.kicad_pcb, SqueezeAMPagain.kicad_prl, SqueezeAMPagain.kicad_pro, and 11 more files
Other:
- title: (none) -> SqueezeAMP_{again}
- moved on the sheet: TP10, TP5, TP6, TP7, TP8, TP9

Commit message: Update SqueezeAMPagain.kicad_pcb, SqueezeAMPagain.kicad_prl, SqueezeAMPagain.kicad_pro, and 4 more files
Parts:
- added R48: 10k, Resistor_SMD:R_0603_1608Metric, symbol Device:R
Connections:
- net +3.3V: now also R48.1
- net Amp/~{SPK_MUTE}: now also R48.2
Changed lines of the file:
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@@
 	)
 	(junction
+		(at 208.28 77.47)
+		(diameter 0)
+		(color 0 0 0 0)
+	)
+	(junction
 		(at 78.74 100.33)
 		(diameter 0)
@@
 	(wire
 		(pts
-			(xy 158.75 77.47) (xy 226.06 77.47)
+			(xy 158.75 77.47) (xy 208.28 77.47)
 		)
 		(stroke
@@
 	(wire
 		(pts
+			(xy 208.28 71.12) (xy 208.28 77.47)
+		)
+		(stroke
+			(width 0)
+			(type default)
+		)
+	)
+	(wire
+		(pts
 			(xy 50.8 85.09) (xy 59.69 85.09)
 		)
@@
 	(wire
 		(pts
+			(xy 208.28 77.47) (xy 226.06 77.47)
+		)
+		(stroke
+			(width 0)
+			(type default)
+		)
+	)
+	(wire
+		(pts
 			(xy 50.8 80.01) (xy 53.34 80.01)
 		)
@@
 	)
 	(symbol
+		(lib_id "power:+3.3V")
+		(at 208.28 63.5 0)
+		(unit 1)
+		(exclude_from_sim no)
+		(in_bom yes)
+		(on_board yes)
+		(dnp no)
+		(fields_autoplaced yes)
+		(property "Reference" "#PWR03"
+			(at 208.28 67.31 0)
+			(effects
+				(font
+					(size 1.27 1.27)
+				)
+				(hide yes)
+			)
+		)
+		(property "Value" "+3.3V"
+			(at 208.28 58.42 0)
+			(effects
+				(font
+					(size 1.27 1.27)
+				)
+			)
+		)
+		(property "Footprint" ""
+			(at 208.28 63.5 0)
+			(effects
+				(font
+					(size 1.27 1.27)
+				)
+				(hide yes)
+			)
+		)
+		(property "Datasheet" ""
+			(at 208.28 63.5 0)
+			(effects
+				(font
+					(size 1.27 1.27)
+				)
+				(hide yes)
+			)
+		)
+		(property "Description" "Power symbol creates a global label with name \"+3.3V\""
+			(at 208.28 63.5 0)
+			(effects
+				(font
+					(size 1.27 1.27)
+				)
+				(hide yes)
+			)
+		)
+		(pin "1"
+		)
+		(instances
+			(project "SqueezeAMPagain"
+				(path "/3675160b-d9e5-490e-b506-2a7966e79ed0"
+					(reference "#PWR03")
+					(unit 1)
+				)
+			)
+		)
+	)
+	(symbol
 		(lib_id "Connector:TestPoint")
 		(at 269.24 55.88 270)
@@
 					(unit 1)
 				)
+			)
+		)
+	)
+	(symbol
+		(lib_id "Device:R")
+		(at 208.28 67.31 0)
+		(unit 1)
+		(exclude_from_sim no)
+		(in_bom yes)
+		(on_board yes)
+		(dnp no)
+		(property "Reference" "R48"
+			(at 210.82 66.0399 0)
+			(effects
+				(font
+					(size 1.27 1.27)
+				)
+				(justify left)
+			)
+		)
+		(property "Value" "10k"
+			(at 210.82 68.5799 0)
+			(effects
+				(font
+					(size 1.27 1.27)
+				)
+				(justify left)
+			)
+		)
+		(property "Footprint" "Resistor_SMD:R_0603_1608Metric"
+			(at 206.502 67.31 90)
+			(effects
+				(font
+					(size 1.27 1.27)
+				)
+				(hide yes)
+			)
+		)
+		(property "Datasheet" "~"
+			(at 208.28 67.31 0)
+			(effects
+				(font
+					(size 1.27 1.27)
+				)
+				(hide yes)
+			)
+		)
+		(property "Description" "Resistor"
+			(at 208.28 67.31 0)
+			(effects
+				(font
+					(size 1.27 1.27)
+				)
+				(hide yes)
+			)
+		)
+		(property "JLCPCB#" "C25804"
+			(at 208.28 67.31 0)
+			(effects
+				(font
+					(size 1.27 1.27)
+				)
+				(hide yes)
+			)
+		)
+		(pin "1"
+		)
+		(pin "2"
+		)
+		(instances
+			(project "SqueezeAMPagain"
+				(path "/3675160b-d9e5-490e-b506-2a7966e79ed0"
+					(reference "R48")
+					(unit 1)
+				)

Commit message: shrink
Parts:
- removed TP5: Mclk, TestPoint:TestPoint_Pad_D1.0mm, symbol Connector:TestPoint
- R2, R3: footprint Resistor_SMD:R_0603_1608Metric -> Resistor_SMD:R_0402_1005Metric
- R48: footprint Resistor_SMD:R_0603_1608Metric -> Resistor_SMD:R_0402_1005Metric; now not fitted
Connections:
- net Amp/MCLK: no longer names the net of R1.2
Other:
- removed sheet Pi
- removed sheet Pico
- sheet Amp ports: added none; removed MCLK
- sheet Power ports: added none; removed LV_ON

Commit message: v2
Parts:
- removed R1: 33, Resistor_SMD:R_0402_1005Metric, symbol Device:R
- removed TP2: 3V3_{SW}, TestPoint:TestPoint_Pad_D1.0mm, symbol Connector:TestPoint
- added SW2: SW_MEC_5G, Button_Switch_SMD:SW_Push_1P1T_XKB_TS-1187A, symbol Switch:SW_MEC_5G
- renumbered R48 to R1, TP6 to TP1, TP11 to TP10, TP12 to TP11, TP7 to TP2, TP8 to TP3, TP9 to TP4, TP10 to TP5, TP1 to TP6, TP3 to TP8, TP4 to TP9
Connections:
- net FPConnector/~{WAKE}: now also SW2.3 (B), SW2.4 (B)
- net GND: now also SW2.1 (A), SW2.2 (A)
Other:
- removed sheet X_PSU
- sheet FPConnector ports: added IO5, IO6; removed none
- sheet Power ports: added none; removed PON, ~{WAKE_DETECT}, ~{WAKE}
- sheet esp ports: added GPIO0/BOOT; removed GPIO0/BOOT/I2S0_MCLK

Commit message: v2
Other:
- note added: "Use Boot0 for Switch?"
Changed lines of the file:
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@@
 (kicad_sch
-	(version 20231120)
+	(version 20250114)
 	(generator "eeschema")
-	(generator_version "8.0")
+	(generator_version "9.0")
 	(paper "A4")
 	(title_block
@@
 		(comment 1 "Overview")
 	)
+	(text "M3 x 4:"
+		(exclude_from_sim no)
+		(at 17.272 24.892 0)
+		(effects
+			(font
+				(size 1.27 1.27)
+			)
+		)
+	)
+	(text "Use Boot0 for Switch?"
+		(exclude_from_sim no)
+		(at 50.546 150.368 0)
+		(effects
+			(font
+				(size 1.27 1.27)
+			)
+		)
+	)
+	(text "Heat spreader M2:"
+		(exclude_from_sim no)
+		(at 22.098 55.626 0)
+		(effects
+			(font
+				(size 1.27 1.27)
+			)
+		)
+	)
 	(junction
 		(at 187.96 86.36)
@@
 		)
 	)
-	(text "M3 x 4:"
-		(exclude_from_sim no)
-		(at 17.272 24.892 0)
-		(effects
-			(font
-				(size 1.27 1.27)
-			)
-		)
-	)
-	(text "Heat spreader M2:"
-		(exclude_from_sim no)
-		(at 22.098 55.626 0)
-		(effects
-			(font
-				(size 1.27 1.27)
-			)
-		)
-	)
 	(label "SCL"
 		(at 45.72 123.19 180)
@@
 		(at 226.06 74.93)
 		(size 26.67 35.56)
+		(exclude_from_sim no)
+		(in_bom yes)
+		(on_board yes)
+		(dnp no)
 		(fields_autoplaced yes)
 		(stroke
@@
 		(at 22.86 175.26)
 		(size 25.4 13.97)
+		(exclude_from_sim no)
+		(in_bom yes)
+		(on_board yes)
+		(dnp no)
 		(fields_autoplaced yes)
 		(stroke
@@
 		(at 257.81 74.93)
 		(size 17.78 27.94)
+		(exclude_from_sim no)
+		(in_bom yes)
+		(on_board yes)
+		(dnp no)
 		(fields_autoplaced yes)
 		(stroke
@@
 		(at 129.54 74.93)
 		(size 29.21 57.15)
+		(exclude_from_sim no)
+		(in_bom yes)
+		(on_board yes)
+		(dnp no)
 		(stroke
 			(width 0.1524)
@@
 		(at 38.1 74.93)
 		(size 12.7 12.7)
+		(exclude_from_sim no)
+		(in_bom yes)
+		(on_board yes)
+		(dnp no)
 		(fields_autoplaced yes)
 		(stroke
@@
 		(at 21.59 87.63)
 		(size 12.7 44.45)
+		(exclude_from_sim no)
+		(in_bom yes)
+		(on_board yes)
+		(dnp no)
 		(fields_autoplaced yes)
 		(stroke
@@
 		)
 	)
+	(embedded_fonts no)
 )
