File: SqueezeAMPagain/USB-Uart.kicad_sch (KiCad schematic)
At the start: 19 parts, among them J8 USB_B_Micro, J9 Conn_01x06_Pin, Q8 Q_NPN_BEC, Q9 Q_NPN_BEC, U7 CP2102N-Axx-xQFN28

Commit message: shrink
Parts:
- C83, C84, C87, C88: footprint Capacitor_SMD:C_0603_1608Metric -> Capacitor_SMD:C_0402_1005Metric
- R35, R36, R37, R38, R39: footprint Resistor_SMD:R_0603_1608Metric -> Resistor_SMD:R_0402_1005Metric
Changed lines of the file:
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@@
 			)
 		)
-		(property "Footprint" "Resistor_SMD:R_0603_1608Metric"
+		(property "Footprint" "Resistor_SMD:R_0402_1005Metric"
 			(at 176.53 86.868 90)
 			(effects
@@
 			)
 		)
-		(property "Footprint" "Capacitor_SMD:C_0603_1608Metric"
+		(property "Footprint" "Capacitor_SMD:C_0402_1005Metric"
 			(at 60.6552 120.65 0)
 			(effects
@@
 			)
 		)
-		(property "Footprint" "Resistor_SMD:R_0603_1608Metric"
+		(property "Footprint" "Resistor_SMD:R_0402_1005Metric"
 			(at 90.17 64.008 90)
 			(effects
@@
 			)
 		)
-		(property "Footprint" "Resistor_SMD:R_0603_1608Metric"
+		(property "Footprint" "Resistor_SMD:R_0402_1005Metric"
 			(at 90.17 67.818 90)
 			(effects
@@
 			)
 		)
-		(property "Footprint" "Capacitor_SMD:C_0603_1608Metric"
+		(property "Footprint" "Capacitor_SMD:C_0402_1005Metric"
 			(at 120.3452 48.26 0)
 			(effects
@@
 			)
 		)
-		(property "Footprint" "Capacitor_SMD:C_0603_1608Metric"
+		(property "Footprint" "Capacitor_SMD:C_0402_1005Metric"
 			(at 135.5852 49.53 0)
 			(effects
@@
 			)
 		)
-		(property "Footprint" "Resistor_SMD:R_0603_1608Metric"
+		(property "Footprint" "Resistor_SMD:R_0402_1005Metric"
 			(at 103.378 87.63 90)
 			(effects
@@
 			)
 		)
-		(property "Footprint" "Capacitor_SMD:C_0603_1608Metric"
+		(property "Footprint" "Capacitor_SMD:C_0402_1005Metric"
 			(at 20.0152 104.14 0)
 			(effects
@@
 			)
 		)
-		(property "Footprint" "Resistor_SMD:R_0603_1608Metric"
+		(property "Footprint" "Resistor_SMD:R_0402_1005Metric"
 			(at 176.53 66.548 90)
 			(effects

Commit message: v2
Parts:
- removed J9: Conn_01x06_Pin, Connector_PinHeader_2.54mm:PinHeader_1x06_P2.54mm_Vertical, symbol Connector:Conn_01x06_Pin
- added D3: B5819W, Diode_SMD:D_SOD-123, symbol Device:D_Schottky
- added JP13: SolderJumper_2_Open, Jumper:SolderJumper-2_P1.3mm_Open_RoundedPad1.0x1.5mm, symbol Jumper:SolderJumper_2_Open
- added R26: 10R, Resistor_SMD:R_1206_3216Metric_Pad1.30x1.75mm_HandSolder, symbol Device:R
- renumbered C83 to C81, C84 to C82, C85 to C83, C86 to C84, C87 to C85, C88 to C86, C89 to C87, D3 to D6, FB6 to FB5, J8 to J7, Q8 to Q4, Q9 to Q5, R35 to R21, R36 to R22, R37 to R23, R38 to R24, R39 to R25, U7 to U6
Connections:
- net at D6.2 (A), J7.1 (VBUS): now also D3.2 (A)
- new net: JP13.1 (A), R26.1
- new net: D3.1 (K), JP13.2 (B)
- new net PVDD: R26.2
Other:
- moved on the sheet: C82, C83, C84, C85, C86, C87, D6, FB5, Q4, Q5, R21, R22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

Commit message: wip
Changed lines of the file:
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@@
-	)
-	(junction
-		(at 194.31 64.77)
-		(diameter 0)
-		(color 0 0 0 0)
 	)
 	(junction
@@
 	)
 	(junction
+		(at 190.5 64.77)
+		(diameter 0)
+		(color 0 0 0 0)
+	)
+	(junction
 		(at 104.14 66.04)
 		(diameter 0)
@@
 	(wire
 		(pts
+			(xy 190.5 64.77) (xy 196.85 64.77)
+		)
+		(stroke
+			(width 0)
+			(type default)
+		)
+	)
+	(wire
+		(pts
 			(xy 29.21 76.2) (xy 138.43 76.2)
 		)
@@
 	(wire
 		(pts
-			(xy 194.31 64.77) (xy 196.85 64.77)
-		)
-		(stroke
-			(width 0)
-			(type default)
-		)
-	)
-	(wire
-		(pts
 			(xy 215.9 90.17) (xy 215.9 97.79)
 		)
@@
 	(wire
 		(pts
-			(xy 215.9 97.79) (xy 194.31 97.79)
+			(xy 215.9 97.79) (xy 190.5 97.79)
 		)
 		(stroke
@@
 	(wire
 		(pts
-			(xy 194.31 64.77) (xy 194.31 97.79)
+			(xy 190.5 64.77) (xy 190.5 97.79)
 		)
 		(stroke
@@
 	(wire
 		(pts
-			(xy 167.64 64.77) (xy 194.31 64.77)
-		)
-		(stroke
+			(xy 167.64 64.77) (xy 190.5 64.77)
+		)
+		(stroke

Commit message: v2
Other:
- moved on the sheet: D6, FB5, J7
