File: SqueezeAMPagain/esp.kicad_sch (KiCad schematic)
At the start: 5 parts, among them J4 Conn_01x06_Pin, U4 ESP32-WROVER-E

Commit message: Update .gitignore, L_Radial_D12.0mm_P5+6+7.00mm_Fastron_11P.kicad_mod, SqueezeAMPagain.kicad_pcb, and 13 more files
Parts:
- added R22, R23, R24, R25, R26: 33, Resistor_SMD:R_0402_1005Metric, symbol Device:R
- C40: footprint Capacitor_SMD:C_0603_1608Metric -> Capacitor_SMD:C_0805_2012Metric
- J4: footprint Connector_PinHeader_2.54mm:PinHeader_1x06_P2.54mm_Horizontal -> Connector_PinHeader_2.54mm:PinHeader_1x06_P2.54mm_Vertical
Connections:
- net IO34: now also U4.6 (GPIO34/ADC1_CH6)
- net IO35: now also U4.7 (GPIO35/ADC1_CH7)
- net IO36: now also U4.4 (SENSOR_VP/GPIO36/ADC1_CH0)
- net IO39: now also U4.5 (SENSOR_VN/GPIO39/ADC1_CH3)
- net IO27: now reaches U4.12 (ADC2_CH7/GPIO27)
- net +3V3 renamed +3.3V
- net GPIO0/BOOT: no longer names the net of U4.25 (GPIO0/BOOT/ADC2_CH1)
- net GPIO0/BOOT: now also R25.1
- net I2S-CLK: no longer names the net of U4.9 (32K_XN/GPIO33/ADC1_CH5)
- net I2S-CLK: now also R23.2
- net I2S-SD: no longer names the net of U4.8 (32K_XP/GPIO32/ADC1_CH4)
- net I2S-SD: now also R22.2
- net I2S-WS: no longer names the net of U4.10 (DAC_1/ADC2_CH8/GPIO25)
- net I2S-WS: now also R24.1
- net SPDIF_OUT renamed TDO
- net TDO: now also R26.2
- net TCK renamed IO13
- net TDI renamed IO12
- new net GPIO0/BOOT/I2S0_MCLK: R25.2
- new net I2S0_SCLK: R23.1
- new net I2S0_SD: R22.1
- new net I2S0_WCLK: R24.2
- new net IO15: R26.1

Commit message: Update SqueezeAMPagain.kicad_pcb, SqueezeAMPagain.kicad_sch, USB-Uart.kicad_sch, and 4 more files
Parts:
- R22, R23, R24, R25, R26: JLCPCB (none) -> C25105
Changed lines of the file:
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@@
+			)
+		)
+		(property "JLCPCB" "C25105"
+			(at 74.93 77.47 90)
+			(effects
+				(font
+					(size 1.27 1.27)
+				)
+				(hide yes)
 			)
 		)
@@
 			)
 		)
+		(property "JLCPCB" "C25105"
+			(at 60.96 90.17 90)
+			(effects
+				(font
+					(size 1.27 1.27)
+				)
+				(hide yes)
+			)
+		)
 		(pin "1"
 		)
@@
 			)
 		)
+		(property "JLCPCB" "C25105"
+			(at 237.49 100.33 90)
+			(effects
+				(font
+					(size 1.27 1.27)
+				)
+				(hide yes)
+			)
+		)
 		(pin "1"
 		)
@@
 			)
 		)
+		(property "JLCPCB" "C25105"
+			(at 237.49 77.47 90)
+			(effects
+				(font
+					(size 1.27 1.27)
+				)
+				(hide yes)
+			)
+		)
 		(pin "1"
 		)
@@
 			(effects
 				(font
+					(size 1.27 1.27)
+				)
+				(hide yes)
+			)
+		)
+		(property "JLCPCB" "C25105"
+			(at 66.04 74.93 90)
+			(effects
+				(font

Commit message: Update SqueezeAMPagain.kicad_pcb, SqueezeAMPagain.kicad_prl, SqueezeAMPagain.kicad_pro, and 11 more files
Parts:
- renumbered C22 to C54, C40 to C55, J4 to J3, R22 to R10, R23 to R11, R1 to R12, R25 to R13, R24 to R14, R26 to R9, U4 to U2
Changed lines of the file:
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@@
 		(dnp no)
 		(fields_autoplaced yes)
-		(property "Reference" "#PWR062"
+		(property "Reference" "#PWR058"
 			(at 114.3 39.37 0)
 			(effects
@@
 			(project "SqueezeAMPagain"
 				(path "/3675160b-d9e5-490e-b506-2a7966e79ed0/7add08aa-332a-4b28-a3d6-ce8f466a0a0b"
-					(reference "#PWR062")
+					(reference "#PWR058")
 					(unit 1)
 				)
@@
 		(dnp no)
 		(fields_autoplaced yes)
-		(property "Reference" "#PWR012"
+		(property "Reference" "#PWR063"
 			(at 163.83 116.84 0)
 			(effects
@@
 			(project "SqueezeAMPagain"
 				(path "/3675160b-d9e5-490e-b506-2a7966e79ed0/7add08aa-332a-4b28-a3d6-ce8f466a0a0b"
-					(reference "#PWR012")
+					(reference "#PWR063")
 					(unit 1)
 				)
@@
 		(dnp no)
 		(fields_autoplaced yes)
-		(property "Reference" "R23"
+		(property "Reference" "R11"
 			(at 74.93 71.12 90)
 			(effects
@@
 			(project "SqueezeAMPagain"
 				(path "/3675160b-d9e5-490e-b506-2a7966e79ed0/7add08aa-332a-4b28-a3d6-ce8f466a0a0b"
-					(reference "R23")
+					(reference "R11")
 					(unit 1)
 				)
@@
 		(dnp no)
 		(fields_autoplaced yes)
-		(property "Reference" "R26"
+		(property "Reference" "R9"
 			(at 60.96 83.82 90)
 			(effects
@@
 			(project "SqueezeAMPagain"
 				(path "/3675160b-d9e5-490e-b506-2a7966e79ed0/7add08aa-332a-4b28-a3d6-ce8f466a0a0b"
-					(reference "R26")
+					(reference "R9")
 					(unit 1)
 				)
@@
 		(dnp no)
 		(fields_autoplaced yes)
-		(property "Reference" "#PWR064"
+		(property "Reference" "#PWR060"
 			(at 129.54 39.37 0)
 			(effects
@@
 			(project "SqueezeAMPagain"
 				(path "/3675160b-d9e5-490e-b506-2a7966e79ed0/7add08aa-332a-4b28-a3d6-ce8f466a0a0b"
-					(reference "#PWR064")
+					(reference "#PWR060")
 					(unit 1)
 				)
@@
 		(dnp no)
 		(fields_autoplaced yes)
-		(property "Reference" "#PWR08"
+		(property "Reference" "#PWR055"
 			(at 95.25 135.89 0)
 			(effects
@@
 			(project "SqueezeAMPagain"
 				(path "/3675160b-d9e5-490e-b506-2a7966e79ed0/7add08aa-332a-4b28-a3d6-ce8f466a0a0b"
-					(reference "#PWR08")
+					(reference "#PWR055")
 					(unit 1)
 				)
@@
 		(on_board yes)
 		(dnp no)
-		(property "Reference" "R1"
+		(property "Reference" "R12"
 			(at 107.95 62.2299 0)
 			(effects
@@
 			(project "SqueezeAMPagain"
 				(path "/3675160b-d9e5-490e-b506-2a7966e79ed0/7add08aa-332a-4b28-a3d6-ce8f466a0a0b"
-					(reference "R1")
+					(reference "R12")
 					(unit 1)
 				)
@@
 		(dnp no)
 		(fields_autoplaced yes)
-		(property "Reference" "#PWR010"
+		(property "Reference" "#PWR056"
 			(at 105.41 62.23 0)
 			(effects
@@
 			(project "SqueezeAMPagain"
 				(path "/3675160b-d9e5-490e-b506-2a7966e79ed0/7add08aa-332a-4b28-a3d6-ce8f466a0a0b"
-					(reference "#PWR010")
+					(reference "#PWR056")
 					(unit 1)
 				)
@@
 		(dnp no)
 		(fields_autoplaced yes)
-		(property "Reference" "J4"
+		(property "Reference" "J3"
 			(at 69.215 107.95 0)
 			(effects
@@
 			(project "SqueezeAMPagain"
 				(path "/3675160b-d9e5-490e-b506-2a7966e79ed0/7add08aa-332a-4b28-a3d6-ce8f466a0a0b"
-					(reference "J4")
+					(reference "J3")
 					(unit 1)
 				)
@@
 		(dnp no)
 		(fields_autoplaced yes)
-		(property "Reference" "U4"
+		(property "Reference" "U2"
 			(at 163.4841 62.23 0)
 			(effects
@@
 			(project "SqueezeAMPagain"
 				(path "/3675160b-d9e5-490e-b506-2a7966e79ed0/7add08aa-332a-4b28-a3d6-ce8f466a0a0b"
-					(reference "U4")
+					(reference "U2")
 					(unit 1)
 				)
@@
 		(dnp no)
 		(fields_autoplaced yes)
-		(property "Reference" "#PWR014"
+		(property "Reference" "#PWR062"
 			(at 161.29 116.84 0)
 			(effects
@@
 			(project "SqueezeAMPagain"
 				(path "/3675160b-d9e5-490e-b506-2a7966e79ed0/7add08aa-332a-4b28-a3d6-ce8f466a0a0b"
-					(reference "#PWR014")
+					(reference "#PWR062")
 					(unit 1)
 				)
@@
 		(dnp no)
 		(fields_autoplaced yes)
-		(property "Reference" "#PWR065"
+		(property "Reference" "#PWR054"
 			(at 91.44 123.19 0)
 			(effects
@@
 			(project "SqueezeAMPagain"
 				(path "/3675160b-d9e5-490e-b506-2a7966e79ed0/7add08aa-332a-4b28-a3d6-ce8f466a0a0b"
-					(reference "#PWR065")
+					(reference "#PWR054")
 					(unit 1)
 				)
@@
 		(dnp no)
 		(fields_autoplaced yes)
-		(property "Reference" "R24"
+		(property "Reference" "R14"
 			(at 237.49 93.98 90)
 			(effects
@@
 			(project "SqueezeAMPagain"
 				(path "/3675160b-d9e5-490e-b506-2a7966e79ed0/7add08aa-332a-4b28-a3d6-ce8f466a0a0b"
-					(reference "R24")
+					(reference "R14")
 					(unit 1)
 				)
@@
 		(dnp no)
 		(fields_autoplaced yes)
-		(property "Reference" "C22"
+		(property "Reference" "C54"
 			(at 118.11 27.9399 0)
 			(effects
@@
 			(project "SqueezeAMPagain"
 				(path "/3675160b-d9e5-490e-b506-2a7966e79ed0/7add08aa-332a-4b28-a3d6-ce8f466a0a0b"
-					(reference "C22")
+					(reference "C54")
 					(unit 1)
 				)
@@
 		(dnp no)
 		(fields_autoplaced yes)
-		(property "Reference" "#PWR063"
+		(property "Reference" "#PWR059"
 			(at 129.54 29.21 0)
 			(effects
@@
 			(project "SqueezeAMPagain"
 				(path "/3675160b-d9e5-490e-b506-2a7966e79ed0/7add08aa-332a-4b28-a3d6-ce8f466a0a0b"
-					(reference "#PWR063")
+					(reference "#PWR059")
 					(unit 1)
 				)
@@
 		(dnp no)
 		(fields_autoplaced yes)
-		(property "Reference" "R25"
+		(property "Reference" "R13"
 			(at 237.49 71.12 90)
 			(effects
@@
 			(project "SqueezeAMPagain"
 				(path "/3675160b-d9e5-490e-b506-2a7966e79ed0/7add08aa-332a-4b28-a3d6-ce8f466a0a0b"
-					(reference "R25")
+					(reference "R13")
 					(unit 1)
 				)
@@
 		(dnp no)
 		(fields_autoplaced yes)
-		(property "Reference" "#PWR061"
+		(property "Reference" "#PWR057"
 			(at 114.3 29.21 0)
 			(effects
@@
 			(project "SqueezeAMPagain"
 				(path "/3675160b-d9e5-490e-b506-2a7966e79ed0/7add08aa-332a-4b28-a3d6-ce8f466a0a0b"
-					(reference "#PWR061")
+					(reference "#PWR057")
 					(unit 1)
 				)
@@
 		(dnp no)
 		(fields_autoplaced yes)
-		(property "Reference" "R22"
+		(property "Reference" "R10"
 			(at 66.04 68.58 90)
 			(effects
@@
 			(project "SqueezeAMPagain"
 				(path "/3675160b-d9e5-490e-b506-2a7966e79ed0/7add08aa-332a-4b28-a3d6-ce8f466a0a0b"
-					(reference "R22")
+					(reference "R10")
 					(unit 1)
 				)
@@
 		(dnp no)
 		(fields_autoplaced yes)
-		(property "Reference" "C40"
+		(property "Reference" "C55"
 			(at 133.35 27.9399 0)
 			(effects
@@
 			(project "SqueezeAMPagain"
 				(path "/3675160b-d9e5-490e-b506-2a7966e79ed0/7add08aa-332a-4b28-a3d6-ce8f466a0a0b"
-					(reference "C40")
+					(reference "C55")
 					(unit 1)
 				)
@@
 		(dnp no)
 		(fields_autoplaced yes)
-		(property "Reference" "#PWR072"
+		(property "Reference" "#PWR061"
 			(at 161.29 68.58 0)
 			(effects
@@
 			(project ""
 				(path "/3675160b-d9e5-490e-b506-2a7966e79ed0/7add08aa-332a-4b28-a3d6-ce8f466a0a0b"
-					(reference "#PWR072")
-					(unit 1)
-				)
+					(reference "#PWR061")
+					(unit 1)
+				)

Commit message: Update Readme.md and esp.kicad_sch
Other:
- title: (none) -> SqueezeAMP_{again}
Changed lines of the file:
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@@
 	(generator_version "8.0")
 	(paper "A4")
+	(title_block
+		(title "SqueezeAMP_{again}")
+		(date "2024-08-23")
+		(rev "1.0")
+	)
 	(junction
 		(at 105.41 69.85)
@@
 		)
 	)
+	(text_box "\"ESP32-WROVER-E comes with a PCB antenna, and ESP32-WROVER-IE with a connector for an external\nantenna.\""
+		(exclude_from_sim no)
+		(at 134.62 123.19 0)
+		(size 55.88 7.62)
+		(stroke
+			(width 0)
+			(type default)
+		)
+		(fill
+			(type none)
+		)
+		(effects
+			(font
+				(size 1.27 1.27)
+			)
+			(justify left top)
+			(href "https://www.espressif.com/sites/default/files/documentation/esp32-wrover-e_esp32-wrover-ie_datasheet_en.pdf")
+		)
+	)

Commit message: Update SqueezeAMPagain.kicad_pcb, SqueezeAMPagain.kicad_prl, SqueezeAMPagain.kicad_pro, and 4 more files
Parts:
- added R32: 10k, Resistor_SMD:R_0603_1608Metric, symbol Device:R
Connections:
- net +3.3V: now also R32.1
- net at R13.1, U2.25 (GPIO0/BOOT/ADC2_CH1): now also R32.2
Changed lines of the file:
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@@
+	)
+	(junction
+		(at 229.87 77.47)
+		(diameter 0)
+		(color 0 0 0 0)
 	)
 	(junction
@@
 	(wire
 		(pts
+			(xy 229.87 68.58) (xy 229.87 77.47)
+		)
+		(stroke
+			(width 0)
+			(type default)
+		)
+	)
+	(wire
+		(pts
 			(xy 196.85 72.39) (xy 215.9 72.39)
 		)
@@
 	(wire
 		(pts
+			(xy 229.87 59.69) (xy 229.87 60.96)
+		)
+		(stroke
+			(width 0)
+			(type default)
+		)
+	)
+	(wire
+		(pts
 			(xy 196.85 69.85) (xy 215.9 69.85)
 		)
@@
 	(wire
 		(pts
+			(xy 229.87 77.47) (xy 196.85 77.47)
+		)
+		(stroke
+			(width 0)
+			(type default)
+		)
+	)
+	(wire
+		(pts
 			(xy 196.85 95.25) (xy 215.9 95.25)
 		)
@@
 	(wire
 		(pts
-			(xy 233.68 77.47) (xy 196.85 77.47)
+			(xy 233.68 77.47) (xy 229.87 77.47)
 		)
 		(stroke
@@
 	(symbol
 		(lib_id "power:+3.3V")
+		(at 229.87 59.69 0)
+		(unit 1)
+		(exclude_from_sim no)
+		(in_bom yes)
+		(on_board yes)
+		(dnp no)
+		(fields_autoplaced yes)
+		(property "Reference" "#PWR0137"
+			(at 229.87 63.5 0)
+			(effects
+				(font
+					(size 1.27 1.27)
+				)
+				(hide yes)
+			)
+		)
+		(property "Value" "+3.3V"
+			(at 229.87 54.61 0)
+			(effects
+				(font
+					(size 1.27 1.27)
+				)
+			)
+		)
+		(property "Footprint" ""
+			(at 229.87 59.69 0)
+			(effects
+				(font
+					(size 1.27 1.27)
+				)
+				(hide yes)
+			)
+		)
+		(property "Datasheet" ""
+			(at 229.87 59.69 0)
+			(effects
+				(font
+					(size 1.27 1.27)
+				)
+				(hide yes)
+			)
+		)
+		(property "Description" "Power symbol creates a global label with name \"+3.3V\""
+			(at 229.87 59.69 0)
+			(effects
+				(font
+					(size 1.27 1.27)
+				)
+				(hide yes)
+			)
+		)
+		(pin "1"
+		)
+		(instances
+			(project "SqueezeAMPagain"
+				(path "/3675160b-d9e5-490e-b506-2a7966e79ed0/7add08aa-332a-4b28-a3d6-ce8f466a0a0b"
+					(reference "#PWR0137")
+					(unit 1)
+				)
+			)
+		)
+	)
+	(symbol
+		(lib_id "power:+3.3V")
 		(at 105.41 58.42 0)
 		(unit 1)
@@
 					(unit 1)
 				)
+			)
+		)
+	)
+	(symbol
+		(lib_id "Device:R")
+		(at 229.87 64.77 0)
+		(unit 1)
+		(exclude_from_sim no)
+		(in_bom yes)
+		(on_board yes)
+		(dnp no)
+		(property "Reference" "R32"
+			(at 232.41 63.4999 0)
+			(effects
+				(font
+					(size 1.27 1.27)
+				)
+				(justify left)
+			)
+		)
+		(property "Value" "10k"
+			(at 232.41 66.0399 0)
+			(effects
+				(font
+					(size 1.27 1.27)
+				)
+				(justify left)
+			)
+		)
+		(property "Footprint" "Resistor_SMD:R_0603_1608Metric"
+			(at 228.092 64.77 90)
+			(effects
+				(font
+					(size 1.27 1.27)
+				)
+				(hide yes)
+			)
+		)
+		(property "Datasheet" "~"
+			(at 229.87 64.77 0)
+			(effects
+				(font
+					(size 1.27 1.27)
+				)
+				(hide yes)
+			)
+		)
+		(property "Description" "Resistor"
+			(at 229.87 64.77 0)
+			(effects
+				(font
+					(size 1.27 1.27)
+				)
+				(hide yes)
+			)
+		)
+		(pin "1"
+		)
+		(pin "2"
+		)
+		(instances
+			(project "SqueezeAMPagain"
+				(path "/3675160b-d9e5-490e-b506-2a7966e79ed0/7add08aa-332a-4b28-a3d6-ce8f466a0a0b"
+					(reference "R32")
+					(unit 1)
+				)

Commit message: shrink
Parts:
- C54: footprint Capacitor_SMD:C_0603_1608Metric -> Capacitor_SMD:C_0402_1005Metric
- R12, R32: footprint Resistor_SMD:R_0603_1608Metric -> Resistor_SMD:R_0402_1005Metric
Changed lines of the file:
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@@
 			)
 		)
-		(property "Footprint" "Resistor_SMD:R_0603_1608Metric"
+		(property "Footprint" "Resistor_SMD:R_0402_1005Metric"
 			(at 103.632 63.5 90)
 			(effects
@@
 			)
 		)
-		(property "Footprint" "Resistor_SMD:R_0603_1608Metric"
+		(property "Footprint" "Resistor_SMD:R_0402_1005Metric"
 			(at 228.092 64.77 90)
 			(effects
@@
 			)
 		)
-		(property "Footprint" "Capacitor_SMD:C_0603_1608Metric"
+		(property "Footprint" "Capacitor_SMD:C_0402_1005Metric"
 			(at 115.2652 33.02 0)
 			(effects

Commit message: v2
Parts:
- removed J3: Conn_01x06_Pin, Connector_PinHeader_2.54mm:PinHeader_1x06_P2.54mm_Vertical, symbol Connector:Conn_01x06_Pin
- added J3: Conn_ARM_JTAG_SWD_10, Connector_PinHeader_1.27mm:PinHeader_2x05_P1.27mm_Vertical_SMD, symbol Connector:Conn_ARM_JTAG_SWD_10
- added R27: 10k, Resistor_SMD:R_0402_1005Metric, symbol Device:R
- renumbered C54 to C56, C55 to C57, R32 to R13, R13 to R14, R14 to R15
Connections:
- net +3.3V: now also J3.1 (VTref), R27.1
- net EN/~{RESET}: now also J3.10 (~{RESET})
- net GND: now also J3.3 (GND), J3.5 (GND), J3.9 (GNDDetect)
- net IO12: now also J3.8 (NC/TDI)
- net IO13: now also J3.4 (SWCLK/TCK)
- net IO15: now also R27.2
- net MUTE: now also J3.2 (SWDIO/TMS)
- net TDO: now also J3.6 (SWO/TDO)
- net GPIO0/BOOT/I2S0_MCLK renamed GPIO0/BOOT
Other:
- moved on the sheet: R9
