File: SqueezeAMPagain/power.kicad_sch (KiCad schematic)
At the start: 86 parts, among them J6 Barrel_Jack_Switch, J7 Conn_01x02_Pin, Q1 Q_NPN_BEC, Q10 AO3401A, Q11 Q_NPN_BEC, Q12 AO3401A, Q13 AO3401A, Q2 AO3401A, Q3 AO3401A, Q4 AO3401A, Q5 Q_NPN_BEC, Q6 AO3401A, Q7 AO3401A, SW1 SW_MEC_5E, U5 AMS1117-3.3, U6 TPS5430DDA

Commit message: Update SqueezeAMPagain.kicad_pcb, SqueezeAMPagain.kicad_prl, SqueezeAMPagain.kicad_pro, and 11 more files
Other:
- title: (none) -> SqueezeAMP_{again}
Changed lines of the file:
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@@
 	(generator_version "8.0")
 	(paper "A4")
+	(title_block
+		(title "SqueezeAMP_{again}")
+		(date "2024-08-23")
+		(rev "1.0")
+	)
 	(junction
 		(at 40.64 63.5)
@@
 		(on_board yes)
 		(dnp no)
-		(fields_autoplaced yes)
 		(property "Reference" "JP11"
 			(at 82.55 13.97 0)

Commit message: Update SqueezeAMPagain.kicad_pcb, SqueezeAMPagain.kicad_prl, SqueezeAMPagain.kicad_pro, and 4 more files
Parts:
- removed C71: 100n, Capacitor_SMD:C_0603_1608Metric, symbol Device:C
- removed R32: 560R, Resistor_SMD:R_0603_1608Metric, symbol Device:R
- added D11: B5819W, Diode_SMD:D_SOD-123, symbol Device:D_Schottky
- added JP15: LV On, Jumper:SolderJumper-2_P1.3mm_Open_RoundedPad1.0x1.5mm, symbol Jumper:SolderJumper_2_Open
Connections:
- net +3.3V: now also JP15.1 (A)
- net +3.3V_{SW}: now also JP15.2 (B)
- net V_{IN}: now also D11.2 (A); no longer FB2.1
- new net: D11.1 (K), FB2.1

Commit message: shrink
Parts:
- removed C90: 2.2u/25V, Capacitor_SMD:C_0805_2012Metric, symbol Device:C
- removed C91: 100n, Capacitor_SMD:C_0603_1608Metric, symbol Device:C
- removed D1: B5819W, Diode_SMD:D_SOD-123, symbol Device:D_Schottky
- removed D10, D9: min. 1.4V_{ff}, LED_SMD:LED_0603_1608Metric, symbol Device:LED
- removed D6, D7: LED, LED_SMD:LED_0603_1608Metric, symbol Device:LED
- removed FB2: 600Ω@100MHz 500mA, Inductor_SMD:L_0805_2012Metric, symbol Device:FerriteBead_Small
- removed JP10, JP15: LV On, Jumper:SolderJumper-2_P1.3mm_Open_RoundedPad1.0x1.5mm, symbol Jumper:SolderJumper_2_Open
- removed JP12: P On, Jumper:SolderJumper-2_P1.3mm_Open_RoundedPad1.0x1.5mm, symbol Jumper:SolderJumper_2_Open
- removed L7: 4.7uH/4.0A, Inductor:L_Radial_D12.0mm_P5+6+7.00mm_Fastron_11P, symbol Device:L_Iron
- removed NT2: NetTie_2, NetTie:NetTie-2_SMD_Pad2.0mm, symbol Device:NetTie_2
- removed Q1, Q11, Q5: Q_NPN_BEC, Package_TO_SOT_SMD:SOT-23, symbol Device:Q_NPN_BEC
- removed Q10, Q12, Q2, Q6, Q7: AO3401A, Package_TO_SOT_SMD:SOT-23, symbol Transistor_FET:AO3401A
- removed R22, R23, R25, R28, R29, R31, R41, R42, R45, R46, R47: 10k, Resistor_SMD:R_0603_1608Metric, symbol Device:R
- removed R24, R30, R40: 150k, Resistor_SMD:R_0603_1608Metric, symbol Device:R
- removed R44: 330, Resistor_SMD:R_0603_1608Metric, symbol Device:R
- removed SW1: SW_MEC_5E, Button_Switch_SMD:SW_Push_1P1T_XKB_TS-1187A, symbol Switch:SW_Push
- C60, C80: footprint Capacitor_SMD:C_0603_1608Metric -> Capacitor_SMD:C_0402_1005Metric
- R33, R34, R43: footprint Resistor_SMD:R_0603_1608Metric -> Resistor_SMD:R_0402_1005Metric
Connections:
- net GND_{IN} is gone; now on net PGND: C66.2, C68.2, NT1.2
- net V_{IN} is gone; now on net PVDD: C66.1, C68.1, D11.2 (A), L5.2
- net at D11.1 (K): now also FB4.1
Other:
- note removed: "Power Switch"
- moved on the sheet: C74, C76, D11

Commit message: v2
Parts:
- removed C74: 100n, Capacitor_SMD:C_0603_1608Metric, symbol Device:C
- removed D8: min. 1.4V_{ff}, LED_SMD:LED_0603_1608Metric, symbol Device:LED
- removed L5: 4.7uH/4.0A, Inductor:L_Radial_D12.0mm_P5+6+7.00mm_Fastron_11P, symbol Device:L_Iron
- added C88: 2.2u/25V, Capacitor_SMD:C_0805_2012Metric, symbol Device:C
- added D7: 5V, Diode_SMD:D_SOD-123, symbol Device:D_Zener
- added L1: 4.7uH/6.0A, Inductor_SMD:L_Chilisin_BMRA00040420, symbol Device:L_Iron
- added L4: 4.7uH/6.0A, Inductor_THT:L_Radial_D8.7mm_P5.00mm_Fastron_07HCP, symbol Device:L_Iron
- C60: renamed from C64; footprint Capacitor_SMD:C_0603_1608Metric -> Capacitor_SMD:C_0402_1005Metric
- C73: footprint Capacitor_SMD:C_0603_1608Metric -> Capacitor_SMD:C_0402_1005Metric
- J5: renamed from J6; footprint Connector_BarrelJack:BarrelJack_CUI_PJ-102AH_Horizontal -> Connector_BarrelJack:BarrelJack_GCT_DCJ200-10-A_Horizontal
- L14: renamed from L6; footprint Inductor_SMD:L_Chilisin_BMRB00060612 -> Inductor_SMD:L_Changjiang_FNR5020S
- R17: renamed from R27; footprint Resistor_SMD:R_0603_1608Metric -> Resistor_SMD:R_0402_1005Metric
- R18: renamed from R43; value 330 -> 1k
- renumbered C59 to C58, C60 to C59, C66 to C63, C63 to C64, C68 to C66, C76 to C69, C69 to C70, C70 to C71, C75 to C74, C77 to C75, C78 to C76, C79 to C77, C80 to C78, C81 to C79, C82 to C80, D4 to D1, D11 to D2, D5 to D4, D2 to D5, FB3 to FB2, FB4 to FB3, FB5 to FB4, J7 to J6, JP11 to JP10, JP13 to JP11, JP14 to JP9, Q13 to Q1, Q3 to Q2, Q4 to Q3, R26 to R16, R33 to R19, R34 to R20, U5 to U4, U6 to U5
Connections:
- net +5V: now also C88.1
- net GND: now also C88.2
- net PVDD: now also L1.2, L4.2; no longer D2.2 (A)
- net V_{supply,plug}: now also D7.1 (K)
- net V_{supply}: now also D2.2 (A), L1.1, L4.1
- net at Q1.1 (G), Q2.1 (G), Q3.1 (G)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: now also D7.2 (A)
Other:
- note removed: "VGS_max ±20 V!"
- moved on the sheet: C59, C60, C61, C62, C64, C65, C67, C70, C71, C72, C73, D4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

Commit message: wip
Parts:
- removed C65: 2.2u/25V, Capacitor_SMD:C_0805_2012Metric, symbol Device:C
Changed lines of the file:
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@@
 	)
 	(junction
-		(at 99.06 118.11)
-		(diameter 0)
-		(color 0 0 0 0)
-	)
-	(junction
 		(at 186.69 134.62)
 		(diameter 0)
@@
 	(wire
 		(pts
-			(xy 99.06 118.11) (xy 113.03 118.11)
+			(xy 93.98 118.11) (xy 113.03 118.11)
 		)
 		(stroke
@@
 	(wire
 		(pts
-			(xy 99.06 118.11) (xy 99.06 130.81)
-		)
-		(stroke
-			(width 0)
-			(type default)
-		)
-	)
-	(wire
-		(pts
 			(xy 78.74 20.32) (xy 71.12 20.32)
 		)
@@
 	(wire
 		(pts
-			(xy 93.98 118.11) (xy 99.06 118.11)
-		)
-		(stroke
-			(width 0)
-			(type default)
-		)
-	)
-	(wire
-		(pts
 			(xy 173.99 63.5) (xy 182.88 63.5)
 		)
@@
 	(wire
 		(pts
-			(xy 99.06 138.43) (xy 99.06 142.24)
-		)
-		(stroke
-			(width 0)
-			(type default)
-		)
-	)
-	(wire
-		(pts
 			(xy 40.64 63.5) (xy 53.34 63.5)
 		)
@@
 	(symbol
 		(lib_id "power:GND")
-		(at 99.06 142.24 0)
-		(unit 1)
-		(exclude_from_sim no)
-		(in_bom yes)
-		(on_board yes)
-		(dnp no)
-		(fields_autoplaced yes)
-		(property "Reference" "#PWR088"
-			(at 99.06 148.59 0)
-			(effects
-				(font
-					(size 1.27 1.27)
-				)
-				(hide yes)
-			)
-		)
-		(property "Value" "GND"
-			(at 99.06 147.32 0)
-			(effects
-				(font
-					(size 1.27 1.27)
-				)
-			)
-		)
-		(property "Footprint" ""
-			(at 99.06 142.24 0)
-			(effects
-				(font
-					(size 1.27 1.27)
-				)
-				(hide yes)
-			)
-		)
-		(property "Datasheet" ""
-			(at 99.06 142.24 0)
-			(effects
-				(font
-					(size 1.27 1.27)
-				)
-				(hide yes)
-			)
-		)
-		(property "Description" "Power symbol creates a global label with name \"GND\" , ground"
-			(at 99.06 142.24 0)
-			(effects
-				(font
-					(size 1.27 1.27)
-				)
-				(hide yes)
-			)
-		)
-		(pin "1"
-		)
-		(instances
-			(project "SqueezeAMPagain"
-				(path "/3675160b-d9e5-490e-b506-2a7966e79ed0/0f57a469-41de-4f06-810e-cfdb6f5b9e50"
-					(reference "#PWR088")
-					(unit 1)
-				)
-			)
-		)
-	)
-	(symbol
-		(lib_id "power:GND")
 		(at 186.69 135.89 0)
 		(unit 1)
@@
 					(unit 1)
 				)
-			)
-		)
-	)
-	(symbol
-		(lib_id "Device:C")
-		(at 99.06 134.62 0)
-		(unit 1)
-		(exclude_from_sim no)
-		(in_bom yes)
-		(on_board yes)
-		(dnp no)
-		(fields_autoplaced yes)
-		(property "Reference" "C65"
-			(at 102.87 133.3499 0)
-			(effects
-				(font
-					(size 1.27 1.27)
-				)
-				(justify left)
-			)
-		)
-		(property "Value" "2.2u/25V"
-			(at 102.87 135.8899 0)
-			(effects
-				(font
-					(size 1.27 1.27)
-				)
-				(justify left)
-			)
-		)
-		(property "Footprint" "Capacitor_SMD:C_0805_2012Metric"
-			(at 100.0252 138.43 0)
-			(effects
-				(font
-					(size 1.27 1.27)
-				)
-				(hide yes)
-			)
-		)
-		(property "Datasheet" "~"
-			(at 99.06 134.62 0)
-			(effects
-				(font
-					(size 1.27 1.27)
-				)
-				(hide yes)
-			)
-		)
-		(property "Description" "Unpolarized capacitor"
-			(at 99.06 134.62 0)
-			(effects
-				(font
-					(size 1.27 1.27)
-				)
-				(hide yes)
-			)
-		)
-		(pin "2"
-		)
-		(pin "1"
-		)
-		(instances
-			(project "SqueezeAMPagain"
-				(path "/3675160b-d9e5-490e-b506-2a7966e79ed0/0f57a469-41de-4f06-810e-cfdb6f5b9e50"
-					(reference "C65")
-					(unit 1)
-				)

Commit message: v2
Parts:
- J5: reichelt# CLIFF FCR681465P -> DC-BU 072759
- L14: jlcpcb C475526 -> C5127240
Other:
- note added: "replace by 0603 for standard components"
Changed lines of the file:
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@@
 (kicad_sch
-	(version 20231120)
+	(version 20250114)
 	(generator "eeschema")
-	(generator_version "8.0")
+	(generator_version "9.0")
 	(paper "A4")
 	(title_block
@@
 		(rev "1.0")
 	)
+	(text "Reverse polarity protection"
+		(exclude_from_sim no)
+		(at 64.008 14.478 0)
+		(effects
+			(font
+				(size 1.27 1.27)
+			)
+		)
+	)
+	(text "\"Float the pin \nto enable.\""
+		(exclude_from_sim no)
+		(at 120.65 133.604 0)
+		(effects
+			(font
+				(size 1.27 1.27)
+			)
+		)
+	)
+	(text "replace by 0603 for standard components"
+		(exclude_from_sim no)
+		(at 225.298 155.956 0)
+		(effects
+			(font
+				(size 1.27 1.27)
+			)
+		)
+	)
+	(text "TI: 549R"
+		(exclude_from_sim no)
+		(at 168.402 161.036 0)
+		(effects
+			(font
+				(size 1.27 1.27)
+			)
+		)
+	)
+	(text "V_{UVLO,typ}  5.3V"
+		(exclude_from_sim no)
+		(at 110.998 112.268 0)
+		(effects
+			(font
+				(size 1.27 1.27)
+			)
+		)
+	)
 	(junction
 		(at 40.64 63.5)
@@
 		)
 	)
-	(text_box "3,3V:\nTI recommendation 10k / 5,9k\nJLC Solution 22k/13k C318507/C22797\n"
-		(exclude_from_sim no)
-		(at 245.11 152.4 0)
-		(size 34.29 12.7)
-		(stroke
-			(width 0)
-			(type default)
-		)
-		(fill
-			(type none)
-		)
-		(effects
-			(font
-				(size 1.27 1.27)
-			)
-			(justify left top)
-		)
-	)
-	(text "Reverse polarity protection"
-		(exclude_from_sim no)
-		(at 64.008 14.478 0)
-		(effects
-			(font
-				(size 1.27 1.27)
-			)
-		)
-	)
-	(text "\"Float the pin \nto enable.\""
-		(exclude_from_sim no)
-		(at 120.65 133.604 0)
-		(effects
-			(font
-				(size 1.27 1.27)
-			)
-		)
-	)
-	(text "TI: 549R"
-		(exclude_from_sim no)
-		(at 168.402 161.036 0)
-		(effects
-			(font
-				(size 1.27 1.27)
-			)
-		)
-	)
-	(text "V_{UVLO,typ}  5.3V"
-		(exclude_from_sim no)
-		(at 110.998 112.268 0)
-		(effects
-			(font
-				(size 1.27 1.27)
-			)
-		)
-	)
 	(label "GND_{supply}"
 		(at 57.15 92.71 0)
@@
 			)
 		)
-		(property "jlcpcb" "C475526"
+		(property "jlcpcb" "C5127240"
 			(at 173.99 123.19 90)
 			(effects
@@
 			)
 		)
-		(property "reichelt#" "CLIFF FCR681465P"
+		(property "reichelt#" "DC-BU 072759"
 			(at 22.86 66.04 0)
 			(effects
