File: SqueezeAMPagain/spkconn.kicad_sch (KiCad schematic)
At the start: 2 parts, among them J1 Conn_01x02_Pin, J2 Conn_01x02_Pin

Commit message: Update SqueezeAMPagain.kicad_pcb, SqueezeAMPagain.kicad_prl, SqueezeAMPagain.kicad_pro, and 11 more files
Other:
- title: (none) -> SqueezeAMP_{again}
Changed lines of the file:
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@@
 	(generator_version "8.0")
 	(paper "A4")
+	(title_block
+		(title "SqueezeAMP_{again}")
+		(date "2024-08-23")
+		(rev "1.0")
+	)
 	(wire
 		(pts
@@
 	(wire
 		(pts
-			(xy 100.33 99.06) (xy 127 99.06)
+			(xy 105.41 99.06) (xy 127 99.06)
 		)
 		(stroke
@@
 	(wire
 		(pts
-			(xy 127 96.52) (xy 101.6 96.52)
+			(xy 127 96.52) (xy 105.41 96.52)
 		)
 		(stroke
@@
 	(hierarchical_label "B-"
 		(shape input)
-		(at 100.33 99.06 180)
+		(at 105.41 99.06 180)
 		(fields_autoplaced yes)
 		(effects
@@
 	(hierarchical_label "B+"
 		(shape input)
-		(at 101.6 96.52 180)
+		(at 105.41 96.52 180)
 		(fields_autoplaced yes)
 		(effects
